File: eagle/regulator_plus_switch.brd (EAGLE design)
At the start: 152.4 x 152.4 mm, 38 parts, among them IC1 LT1352PA, T1 2N3904, T2 2N3904

Commit message: More fixes...and a board with digital in
Parts:
- added IC2, IC4: LT1352PA, linear-technology:DIL08
- added IC3: DG419DJN, linear:DIL08
- added R16, R18, R27, R31: 10k, rcl:0207/10
- added R17, R28: 40k, rcl:0207/10
- added R19, R29: 17k, rcl:0207/10
- added R20, R30: 13k, rcl:0207/10
- added R21, R22, R23, R24, R25: 1M, resistor:0414/15
- added R26: 50k, rcl:0207/10
- added R32: 100k, rcl:0207/10
- added U$4: 5569-2, con-molex:5569-2
- added X2: (no value), con-molex:KK-156-6
- OK1: value CNY17 -> H11F1; device optocoupler:DIL06 -> optocoupler:DIL05
- R12: value 250 -> 10k
- R13, R14: device rcl:0207/10 -> rcl:0207/15
- X1: device con-molex:KK-156-6 -> con-subd:F25HP
- moved C1 128.2 mm to (8.89, 175.3)
- moved U$1 108.5 mm to (14.0, 125.7)
- moved R14 101.3 mm to (31.8, 137.2)
- moved D1 99.2 mm to (132.1, 205.7)
- moved D2 99.2 mm to (142.2, 190.5)
- moved D4 99.2 mm to (142.2, 160.0)
- moved D5 99.2 mm to (132.1, 144.8)
- moved D3 99.2 mm to (132.1, 175.3)
- moved D6 99.2 mm to (142.2, 129.5)
- moved C5 99.1 mm to (29.2, 114.3)
- moved R3 99.1 mm to (96.5, 213.4)
- moved R4 99.1 mm to (81.3, 177.8)
- moved R6 99.1 mm to (76.2, 163.8)
- moved T1 99.1 mm to (99.1, 195.6), flipped to the top
- moved C4 99.1 mm to (61.0, 198.1)
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Connections:
- new net CMD1: R16.2, X1.1
- new net N$24: IC2.2, R16.1, R17.2
- new net N$25: IC2.3, R18.1
- new net N$26: R18.2, R19.2, R20.1
- new net N$27: IC2.1, IC3.8, R17.1
- new net N$28: IC3.1, R10.2
- new net N$29: IC3.6, R32.2, U$4.P$2
- new net N$30: R21.1, R22.2
- new net N$31: R22.1, R23.2
- new net N$32: R23.1, R24.2
- new net N$33: R24.1, R25.2
- new net N$34: R25.1, R26.2, R28.2
- new net N$35: IC4.1, R27.1, X1.17
- new net N$36: R29.2, R30.1, R31.2
- new net N$37: IC4.3, R31.1
- new net N$39: IC4.2, R27.2, R28.1
- net +15V: now also C2.1, IC2.8, IC3.4, IC4.8, R20.2, R30.2, X2.6; no longer C1.1, X1.6
- net +5V: now also IC3.5, U$4.P$1, X2.4, X2.5; no longer X1.4, X1.5
- net -15V: now also C1.1, IC2.4, IC3.7, IC4.4, R19.1, R29.1, X2.1; no longer C2.1, X1.1
- net GND: now also IC3.3, R26.1, R32.1, X1.10, X1.12, X1.14, X1.16, X1.25, X1.4, X1.6, X1.8, X2.2, X2.3; no longer X1.3
- net N$10: now also R21.2
- net N$13: now also IC3.2; no longer R10.2
- net N$16: now also OK1.6; no longer OK1.5
Routing:
- net -15V: track 108.3 -> 222.6 mm, vias 0 -> 2
- net +15V: track 107.9 -> 221.9 mm, vias 0 -> 4
- net +5V: track 0.00 -> 110.4 mm
- net N$34: track 0.00 -> 85.2 mm
- net CMD1: track 0.00 -> 83.4 mm
- net N$13: track 75.3 -> 0.00 mm
- net N$35: track 0.00 -> 66.0 mm
- net N$29: track 0.00 -> 56.6 mm
- net GND: track 2.54 -> 47.3 mm, vias 0 -> 4
- net N$15: track 37.9 -> 0.00 mm
- net N$39: track 0.00 -> 31.6 mm
- net N$36: track 0.00 -> 29.0 mm
- net N$8: track 14.5 -> 40.2 mm, vias 0 -> 2
- net N$18: track 17.8 -> 42.0 mm
- net N$24: track 0.00 -> 23.4 mm
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Other:
- board size 152.4 x 152.4 mm -> 152.4 x 228.6 mm
- board text removed: "2n3904 are on reverse side!!!"

Commit message: multi-channel
Parts:
- added C6: 10n, rcl:C075-032X103
- added D10, D11, D12, D13, D8, D9: P6KEXX, diode:CB417-15
- added D14: 1N4148DO35-10, diode:DO35-10
- added DC2: (no value), dc-dc-converter:NCS
- added IC5, IC6, IC8: LT1352PA, linear-technology:DIL08
- added IC7: DG419DJN, linear:DIL08
- added OK2: CNY17, optocoupler:DIL06
- added Q3, Q4: (no value), transistor-power:TO220BV
- added R33, R34: 65, rcl:0207/10
- added R35, R36: 100, rcl:0207/10
- added R37, R39, R47, R53, R54, R55, R56, R57: 1M, resistor:0414/15
- added R38, R64: 100k, rcl:0207/10
- added R40, R58: 50k, rcl:0207/10
- added R41, R42, R43, R48, R50, R59, R63: 10k, rcl:0207/10
- added R44: 250, rcl:0207/15
- added R45, R46: 20k, rcl:0207/15
- added R49, R60: 40k, rcl:0207/10
- added R51, R61: 17k, rcl:0207/10
- added R52, R62: 13k, rcl:0207/10
- added T3, T4: 2N3904, transistor:TO92
- added U$5: 5569-4, con-molex:5669-4
- added U$6, U$7: 5569-2, con-molex:5569-2
- OK1: value H11F1 -> CNY17; device optocoupler:DIL05 -> optocoupler:DIL06
- R12: value 10k -> 250
- moved OK1 179.9 mm to (-10.4, 6.86), turned to 0 degrees
Connections:
- new net CMD2: R48.2, X1.3
- new net MAN: IC3.6, IC7.6, R32.2, R64.2, U$4.P$2, U$7.P$2
- new net N$38: D10.A, D9.C
- new net N$40: D10.C, D11.C
- new net N$41: D11.A, D12.C
- new net N$42: D12.A, D13.C
- new net N$43: Q3.G, R35.1
- new net N$44: D14.C, Q4.D, R35.2, R37.1, T3.1
- new net N$45: Q3.S, R33.2, T3.2
- new net N$46: D14.A, D8.A, R33.1, R47.2, R53.2, T3.3, U$6.P$1
- new net N$47: Q4.G, R36.1
- new net N$48: OK2.4, R36.2, R38.2, T4.1
- new net N$49: Q4.S, R34.2, T4.2
- new net N$50: DC2.P$6, OK2.5
- new net N$51: C6.1, R41.1
- new net N$52: IC5.2, R41.2, R42.1
- new net N$53: C6.2, IC5.1, R44.2
- new net N$54: IC5.3, R43.1
- new net N$55: R39.1, R40.2, R43.2
- new net N$56: R39.2, R47.1
- new net N$57: IC6.2, R48.1, R49.2
- new net N$58: IC6.3, R50.1
- new net N$59: R50.2, R51.2, R52.1
- new net N$60: IC6.1, IC7.8, R49.1
- new net N$61: IC7.1, R42.2
- new net N$62: R53.1, R54.2
- new net N$63: R54.1, R55.2
- new net N$64: R55.1, R56.2
- new net N$65: R56.1, R57.2
- new net N$66: R57.1, R58.2, R60.2
- new net N$67: IC8.1, R59.1, X1.18
- new net N$68: R61.2, R62.1, R63.2
- new net N$69: IC8.3, R63.1
- new net N$70: IC8.2, R59.2, R60.1
- new net N$71: R45.2, U$5.P$2
- new net N$72: IC7.2, U$5.P$4
- new net N$73: R46.2, U$5.P$1
- new net N$74: OK2.1, R44.1
- net +15V: now also DC2.P$8, DC2.P$9, IC5.8, IC6.8, IC7.4, IC8.8, R45.1, R52.2, R62.2
- net +5V: now also IC7.5, U$7.P$1
- net -15V: now also IC5.4, IC6.4, IC7.7, IC8.4, R46.1, R51.1, R61.1
- net GND: now also D13.A, DC2.P$2, DC2.P$3, IC7.3, OK2.2, R40.1, R58.1, R64.1, U$6.P$2
- net N$16: now also OK1.5; no longer OK1.6
- net N$29: now also D8.C, D9.A; no longer IC3.6, R32.2, U$4.P$2
- net V+: now also Q3.D, R37.2
- net V-: now also DC2.P$7, R34.1, R38.1, T4.3
Routing:
- net N$29: track 56.6 -> 0.00 mm
- net MAN: track 0.00 -> 56.6 mm
- net N$22: track 29.2 -> 0.00 mm
- net N$12: track 35.1 -> 25.0 mm
- net N$16: track 18.1 -> 16.8 mm
