File: eagle/regulator_plus_switch.brd (EAGLE design)
At the start: 152.4 x 152.4 mm, 67 parts, among them IC2 LT1352PA, IC3 DG419DJN, IC4 LT1352PA, Q1 2N3906, Q2 2N3906, T1 2N3904, T2 2N3904

Commit message: overcurrent, worked out connectors
Parts:
- added DISPLAY1, J23: 5569-2, con-molex:5569-2
- added R33: 9.09k, rcl:0207/10
- added R34: 1k, rcl:0207/10
- added R35: 294, rcl:0207/10
- R26: value 5k -> 50k
- R28: value 40k -> 20k
- renumbered GROUND to J26, UNK to J25
Connections:
- new net N$20: DISPLAY1.P$1, R33.2, R34.1
- new net N$21: J23.P$1, R33.1
- new net N$22: J26.P$1, R35.1
- net GND: now also DISPLAY1.P$2, R34.2
- net N$6: now also R35.2; no longer J26.P$1
Routing:
- net N$6: track 15.3 -> 0.36 mm
- net N$34: track 238.8 -> 233.8 mm
Changed lines of the file:
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@@
 <element name="R24" library="resistor" package="0207/10" value="1M" x="124.714" y="49.53" rot="R180"/>
 <element name="R25" library="resistor" package="0207/10" value="1M" x="120.904" y="43.942"/>
-<element name="R26" library="rcl" package="0207/10" value="5k" x="120.904" y="38.608" rot="R180"/>
+<element name="R26" library="rcl" package="0207/10" value="50k" x="120.904" y="38.608" rot="R180"/>
 <element name="IC4" library="linear-technology" package="DIL08" value="LT1352PA" x="46.736" y="28.194">
 <attribute name="OC_NEWARK" value="unknown" x="46.736" y="28.194" size="1.778" layer="27" display="off"/>
@@
 </element>
 <element name="R27" library="rcl" package="0207/10" value="10k" x="50.038" y="9.906" rot="R90"/>
-<element name="R28" library="rcl" package="0207/10" value="40k" x="73.66" y="19.304"/>
+<element name="R28" library="rcl" package="0207/10" value="20k" x="73.66" y="19.304"/>
 <element name="R29" library="rcl" package="0207/10" value="17k" x="45.466" y="20.574" rot="R180"/>
 <element name="R30" library="rcl" package="0207/10" value="13k" x="34.798" y="25.654" rot="R90"/>
@@
 <element name="OUT" library="con-amp-te" package="640584-1" value="640584-1" x="136.906" y="77.216" rot="R270"/>
 <element name="DISPLAY" library="con-molex" package="5669-8" value="5669-8" x="108.204" y="142.494" rot="R180"/>
-<element name="UNK" library="con-molex" package="5569-2" value="5569-2" x="61.468" y="141.478" rot="R180"/>
-<element name="GROUND" library="con-molex" package="5569-2" value="5569-2" x="46.228" y="141.224" rot="R180"/>
+<element name="J25" library="con-molex" package="5569-2" value="5569-2" x="61.468" y="141.478" rot="R180"/>
+<element name="J26" library="con-molex" package="5569-2" value="5569-2" x="46.228" y="141.224" rot="R180"/>
 <element name="DISPLAYPOWER" library="con-molex" package="5569-2" value="5569-2" x="32.004" y="140.716" rot="R180"/>
 <element name="LED" library="con-molex" package="5569-2" value="5569-2" x="80.264" y="141.478" rot="R180"/>
@@
 <element name="C9" library="rcl" package="C075-032X103" value="cc" x="137.16" y="112.268"/>
 <element name="R15" library="rcl" package="0207/10" value="rl" x="134.62" y="106.426"/>
+<element name="DISPLAY1" library="con-molex" package="5569-2" value="5569-2" x="-8.89" y="7.874"/>
+<element name="R33" library="rcl" package="0207/10" value="9.09k" x="-5.334" y="-9.652"/>
+<element name="R34" library="rcl" package="0207/10" value="1k" x="-5.334" y="-14.224"/>
+<element name="J23" library="con-molex" package="5569-2" value="5569-2" x="-17.272" y="-1.27"/>
+<element name="R35" library="rcl" package="0207/10" value="294" x="-13.716" y="-18.796"/>
 </elements>
 <signals>
@@
 <contactref element="POWER" pad="3"/>
 <contactref element="DISPLAYPOWER" pad="P$2"/>
-<contactref element="UNK" pad="P$2"/>
-<contactref element="GROUND" pad="P$2"/>
+<contactref element="J25" pad="P$2"/>
+<contactref element="J26" pad="P$2"/>
 <contactref element="LED" pad="P$2"/>
 <contactref element="D2" pad="A"/>
@@
 <wire x1="54.102" y1="62.484" x2="53.594" y2="62.484" width="1.4224" layer="16"/>
 <wire x1="53.594" y1="62.484" x2="49.784" y2="58.674" width="1.4224" layer="16"/>
+<contactref element="R34" pad="2"/>
+<contactref element="DISPLAY1" pad="P$2"/>
+<wire x1="-8.89" y1="12.192" x2="-0.254" y2="-14.224" width="0" layer="19" extent="1-1"/>
+<wire x1="31.75" y1="58.42" x2="-8.89" y2="12.192" width="0" layer="19" extent="1-1"/>
 </signal>
 <signal name="V+">
@@
 <contactref element="R28" pad="2"/>
 <wire x1="115.824" y1="19.304" x2="78.74" y2="19.304" width="1.4224" layer="16"/>
-<contactref element="DISPLAY" pad="P$1"/>
 <wire x1="115.824" y1="43.942" x2="115.824" y2="67.056" width="1.4224" layer="16"/>
 <wire x1="115.824" y1="67.056" x2="116.586" y2="68.072" width="1.4224" layer="16"/>
@@
 <wire x1="149.606" y1="135.128" x2="138.938" y2="145.796" width="1.4224" layer="16"/>
 <wire x1="138.938" y1="145.796" x2="108.204" y2="145.796" width="1.4224" layer="16"/>
-<wire x1="108.204" y1="145.796" x2="108.204" y2="142.494" width="1.4224" layer="16"/>
-<wire x1="108.204" y1="144.272" x2="108.204" y2="142.494" width="1.4224" layer="16"/>
 <wire x1="115.824" y1="43.942" x2="115.824" y2="38.608" width="1.4224" layer="16"/>
 <wire x1="115.824" y1="43.942" x2="115.824" y2="19.304" width="1.4224" layer="16"/>
+<contactref element="DISPLAY" pad="P$1"/>
+<wire x1="108.204" y1="145.796" x2="108.204" y2="142.494" width="0" layer="19" extent="16-16"/>
 </signal>
 <signal name="N$35">
@@
 </signal>
 <signal name="N$6">
-<contactref element="UNK" pad="P$1"/>
-<contactref element="GROUND" pad="P$1"/>
-<wire x1="46.228" y1="141.224" x2="61.214" y2="141.224" width="1.4224" layer="16"/>
+<contactref element="J25" pad="P$1"/>
 <wire x1="61.214" y1="141.224" x2="61.468" y2="141.478" width="1.4224" layer="16"/>
+<contactref element="R35" pad="2"/>
+<wire x1="-8.636" y1="-18.796" x2="61.214" y2="141.224" width="0" layer="19" extent="16-16"/>
 </signal>
 <signal name="N$7">
@@
 <wire x1="124.968" y1="100.33" x2="123.698" y2="99.06" width="1.4224" layer="16"/>
 </signal>
+<signal name="N$20">
+<contactref element="DISPLAY1" pad="P$1"/>
+<contactref element="R33" pad="2"/>
+<contactref element="R34" pad="1"/>
+<contactref element="R34" pad="1"/>
+<wire x1="-0.254" y1="-9.652" x2="-10.414" y2="-14.224" width="0" layer="19" extent="1-1"/>
+<wire x1="-8.89" y1="7.874" x2="-0.254" y2="-9.652" width="0" layer="19" extent="1-1"/>
+</signal>
+<signal name="N$21">
+<contactref element="R33" pad="1"/>
+<contactref element="J23" pad="P$1"/>
+<wire x1="-17.272" y1="-1.27" x2="-10.414" y2="-9.652" width="0" layer="19" extent="1-1"/>
+</signal>
+<signal name="N$22">
+<contactref element="R35" pad="1"/>
+<contactref element="J26" pad="P$1"/>
+<wire x1="-18.796" y1="-18.796" x2="46.228" y2="141.224" width="0" layer="19" extent="1-1"/>
+</signal>
 </signals>

Commit message: yay led switch worked out
Parts:
- removed J25, LED: 5569-2, con-molex:5569-2
- removed R1: 220, rcl:0207/10
- renumbered DISPLAYPOWER to DISPLAYPOWERJ25
Connections:
- removed net N$6: J25.P$1, R35.2
- removed net N$7: LED.P$1, R1.2
- net +5V: now also R35.2; no longer R1.1
- net GND: no longer J25.P$2, LED.P$2
Routing:
- net +5V: track 297.2 -> 251.2 mm
- net N$7: track 11.4 -> 0.00 mm
Changed lines of the file:
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@@
 <element name="OUT" library="con-amp-te" package="640584-1" value="640584-1" x="136.906" y="77.216" rot="R270"/>
 <element name="DISPLAY" library="con-molex" package="5669-8" value="5669-8" x="108.204" y="142.494" rot="R180"/>
-<element name="J25" library="con-molex" package="5569-2" value="5569-2" x="61.468" y="141.478" rot="R180"/>
 <element name="J26" library="con-molex" package="5569-2" value="5569-2" x="46.228" y="141.224" rot="R180"/>
-<element name="DISPLAYPOWER" library="con-molex" package="5569-2" value="5569-2" x="32.004" y="140.716" rot="R180"/>
-<element name="LED" library="con-molex" package="5569-2" value="5569-2" x="80.264" y="141.478" rot="R180"/>
-<element name="R1" library="rcl" package="0207/10" value="220" x="91.694" y="136.398" rot="R90"/>
+<element name="DISPLAYPOWERJ25" library="con-molex" package="5569-2" value="5569-2" x="32.004" y="140.716" rot="R180"/>
 <element name="D2" library="diode" package="C1702-15" value="P6KEXXA" x="29.21" y="119.38" rot="R90"/>
 <element name="D3" library="diode" package="C1702-15" value="P6KEXXA" x="27.178" y="95.504" rot="R180"/>
@@
 <contactref element="POWER" pad="2"/>
 <contactref element="POWER" pad="3"/>
-<contactref element="DISPLAYPOWER" pad="P$2"/>
-<contactref element="J25" pad="P$2"/>
+<contactref element="DISPLAYPOWERJ25" pad="P$2"/>
 <contactref element="J26" pad="P$2"/>
-<contactref element="LED" pad="P$2"/>
 <contactref element="D2" pad="A"/>
 <contactref element="D3" pad="C"/>
@@
 <contactref element="R34" pad="2"/>
 <contactref element="DISPLAY1" pad="P$2"/>
-<wire x1="-8.89" y1="12.192" x2="-0.254" y2="-14.224" width="0" layer="19" extent="1-1"/>
-<wire x1="31.75" y1="58.42" x2="-8.89" y2="12.192" width="0" layer="19" extent="1-1"/>
+<wire x1="130.302" y1="102.108" x2="139.7" y2="106.426" width="0" layer="19" extent="1-1"/>
+<wire x1="93.98" y1="83.312" x2="130.302" y2="102.108" width="0" layer="19" extent="1-1"/>
+<wire x1="105.664" y1="62.738" x2="93.98" y2="83.312" width="0" layer="19" extent="1-1"/>
+<wire x1="122.2502" y1="12.954" x2="124.46" y2="24.384" width="0" layer="19" extent="16-16"/>
+<wire x1="123.6472" y1="10.414" x2="123.698" y2="10.414" width="0" layer="19" extent="16-16"/>
+<wire x1="118.11" y1="11.5824" x2="122.2502" y2="12.954" width="0" layer="19" extent="16-16"/>
+<wire x1="60.706" y1="53.594" x2="93.98" y2="83.312" width="0" layer="19" extent="1-1"/>
+<wire x1="31.75" y1="66.548" x2="32.004" y2="58.674" width="0" layer="19" extent="16-16"/>
+<wire x1="14.732" y1="74.266" x2="14.732" y2="70.306" width="0" layer="19" extent="1-1"/>
+<wire x1="32.766" y1="78.232" x2="36.068" y2="70.866" width="0" layer="19" extent="16-16"/>
+<wire x1="27.432" y1="90.424" x2="32.766" y2="78.232" width="0" layer="19" extent="1-1"/>
+<wire x1="34.798" y1="95.504" x2="27.432" y2="90.424" width="0" layer="19" extent="1-1"/>
+<wire x1="14.224" y1="101.092" x2="27.432" y2="90.424" width="0" layer="19" extent="1-1"/>
+<wire x1="14.224" y1="105.283" x2="14.224" y2="101.092" width="0" layer="19" extent="1-1"/>
+<wire x1="4.826" y1="113.538" x2="14.224" y2="105.283" width="0" layer="19" extent="16-16"/>
+<wire x1="29.21" y1="127" x2="25.146" y2="132.08" width="0" layer="19" extent="16-16"/>
+<wire x1="19.812" y1="119.38" x2="29.21" y2="127" width="0" layer="19" extent="1-1"/>
+<wire x1="46.228" y1="136.906" x2="32.004" y2="136.398" width="0" layer="19" extent="1-1"/>
+<wire x1="-8.89" y1="12.192" x2="31.75" y2="58.42" width="0" layer="19" extent="1-1"/>
+<wire x1="-0.254" y1="-14.224" x2="-8.89" y2="12.192" width="0" layer="19" extent="1-1"/>
 </signal>
 <signal name="V+">
@@
 <contactref element="POWER" pad="4"/>
 <contactref element="POWER" pad="5"/>
-<contactref element="DISPLAYPOWER" pad="P$1"/>
-<contactref element="R1" pad="1"/>
-<wire x1="91.694" y1="131.318" x2="45.72" y2="131.318" width="1.4224" layer="16"/>
+<contactref element="DISPLAYPOWERJ25" pad="P$1"/>
 <wire x1="45.72" y1="131.318" x2="36.322" y2="140.716" width="1.4224" layer="16"/>
 <wire x1="36.322" y1="140.716" x2="32.512" y2="140.716" width="1.4224" layer="16"/>
@@
 <wire x1="24.638" y1="140.462" x2="32.258" y2="140.462" width="1.4224" layer="16"/>
 <wire x1="32.258" y1="140.462" x2="32.512" y2="140.716" width="1.4224" layer="16"/>
+<contactref element="R35" pad="2"/>
+<wire x1="-8.636" y1="-18.796" x2="18.796" y2="18.034" width="0" layer="19" extent="1-1"/>
 </signal>
 <signal name="N$24">
@@
 <wire x1="10.668" y1="32.512" x2="15.494" y2="27.686" width="1.4224" layer="16"/>
 </signal>
-<signal name="N$6">
-<contactref element="J25" pad="P$1"/>
-<wire x1="61.214" y1="141.224" x2="61.468" y2="141.478" width="1.4224" layer="16"/>
-<contactref element="R35" pad="2"/>
-<wire x1="-8.636" y1="-18.796" x2="61.214" y2="141.224" width="0" layer="19" extent="16-16"/>
-</signal>
-<signal name="N$7">
-<contactref element="LED" pad="P$1"/>
-<contactref element="R1" pad="2"/>
-<wire x1="80.264" y1="141.478" x2="91.694" y2="141.478" width="1.4224" layer="16"/>
-</signal>
 <signal name="N$3">
