File: eagle/regulator_plus_switch.brd (EAGLE design)
At the start: 152.7 x 152.4 mm, 69 parts, among them IC2 LT1352PA, IC3 DG419DJN, IC4 LT1352PA, J23 5569-2, J26 5569-2, Q1 2N3906, Q2 2N3906, T1 2N3904, T2 2N3904

Commit message: 8chan
Parts:
- moved EXTERNAL 116.2 mm to (125.5, -12.7)
