File: eagle/regulator_plus_switch.sch (EAGLE design)
At the start: 38 parts, among them IC1 LT1352PA, T1 2N3904, T2 2N3904

Commit message: More fixes...and a board with digital in
Parts:
- added IC2, IC4: LT1352PA, linear-technology:LT1352PA
- added IC3: DG419DJN, linear:DG419DJN
- added R16, R18, R27, R31: 10k, rcl:R-US_0207/10
- added R17, R28: 40k, rcl:R-US_0207/10
- added R19, R29: 17k, rcl:R-US_0207/10
- added R20, R30: 13k, rcl:R-US_0207/10
- added R21, R22, R23, R24, R25: 1M, resistor:R-US_0414/15
- added R26: 50k, rcl:R-US_0207/10
- added R32: 100k, rcl:R-US_0207/10
- added U$4: 5569-2, con-molex:5569-2
- added X2: (no value), con-molex:KK-156-6
- OK1: value CNY17 -> H11F1; device optocoupler:CNY17 -> optocoupler:H11F1
- R12: value 250 -> 10k
- R13, R14: device rcl:R-US_0207/10 -> rcl:R-US_0207/15
- X1: device con-molex:KK-156-6 -> con-subd:F25HPS
Connections:
- new net CMD1: R16.2, X1-1.F
- new net N$24: IC2A.-IN, R16.1, R17.2
- new net N$25: IC2A.+IN, R18.1
- new net N$26: R18.2, R19.2, R20.1
- new net N$27: IC2A.OUT, IC3A.S2, R17.1
- new net N$28: IC3A.D, R10.2
- new net N$29: IC3A.IN, R32.2, U$4G$2.S
- new net N$30: R21.1, R22.2
- new net N$31: R22.1, R23.2
- new net N$32: R23.1, R24.2
- new net N$33: R24.1, R25.2
- new net N$34: R25.1, R26.2, R28.2
- new net N$35: IC4A.OUT, R27.1, X1-17.F
- new net N$36: R29.2, R30.1, R31.2
- new net N$37: IC4A.+IN, R31.1
- new net N$39: IC4A.-IN, R27.2, R28.1
- net +15V: now also C2.1, IC2A.V+, IC3P.V+, IC4A.V+, R20.2, R30.2, X2-6.S; no longer C1.1, X1-6.S
- net +5V: now also IC3VL.VL, U$4G$1.S, X2-4.S, X2-5.S; no longer X1-4.S, X1-5.S
- net -15V: now also C1.1, IC2A.V-, IC3P.V-, IC4A.V-, R19.1, R29.1, X2-1.S; no longer C2.1, X1-1.S
- net GND: now also IC3P.GND, R26.1, R32.1, X1-10.F, X1-12.F, X1-14.F, X1-16.F, X1-2.F, X1-25.F, X1-4.F, X1-6.F, X1-8.F, X2-2.S, X2-3.S; no longer X1-2.S, X1-3.S
- net N$10: now also R21.2
- net N$12: now also OK1.EMIT; no longer OK1.EMI
- net N$13: now also IC3A.S1; no longer R10.2
Other:
- moved on the sheet: R13, R14, U$1G$1, U$1G$2, U$1G$4, X1-1, X1-2, X1-3, X1-4, X1-5, X1-6

Commit message: multi-channel
Parts:
- added C6: 10n, rcl:C-US075-032X103
- added D10, D11, D12, D13, D8, D9: P6KEXX, diode:P6KEXX
- added D14: 1N4148DO35-10, diode:1N4148DO35-10
- added DC2: (no value), dc-dc-converter:NCS
- added IC5, IC6, IC8: LT1352PA, linear-technology:LT1352PA
- added IC7: DG419DJN, linear:DG419DJN
- added OK2: CNY17, optocoupler:CNY17
- added Q3, Q4: (no value), transistor-power:PMOSFET_NTO220BV
- added R33, R34: 65, rcl:R-US_0207/10
- added R35, R36: 100, rcl:R-US_0207/10
- added R37, R39, R47, R53, R54, R55, R56, R57: 1M, resistor:R-US_0414/15
- added R38, R64: 100k, rcl:R-US_0207/10
- added R40, R58: 50k, rcl:R-US_0207/10
- added R41, R42, R43, R48, R50, R59, R63: 10k, rcl:R-US_0207/10
- added R44: 250, rcl:R-US_0207/15
- added R45, R46: 20k, rcl:R-US_0207/15
- added R49, R60: 40k, rcl:R-US_0207/10
- added R51, R61: 17k, rcl:R-US_0207/10
- added R52, R62: 13k, rcl:R-US_0207/10
- added T3, T4: 2N3904, transistor:2N3904
- added U$5: 5569-4, con-molex:5569-4
- added U$6, U$7: 5569-2, con-molex:5569-2
- OK1: value H11F1 -> CNY17; device optocoupler:H11F1 -> optocoupler:CNY17
- R12: value 10k -> 250
Connections:
- new net CMD2: R48.2, X1-3.F
- new net MAN: IC3A.IN, IC7A.IN, R32.2, R64.2, U$4G$2.S, U$7G$2.S
- new net N$38: D10.A, D9.C
- new net N$40: D10.C, D11.C
- new net N$41: D11.A, D12.C
- new net N$42: D12.A, D13.C
- new net N$43: Q3.G, R35.1
- new net N$44: D14.C, Q4.D, R35.2, R37.1, T3.C
- new net N$45: Q3.S, R33.2, T3.B
- new net N$46: D14.A, D8.A, R33.1, R47.2, R53.2, T3.E, U$6G$1.S
- new net N$47: Q4.G, R36.1
- new net N$48: OK2.EMI, R36.2, R38.2, T4.C
- new net N$49: Q4.S, R34.2, T4.B
- new net N$50: DC2.VOUT, OK2.COL
- new net N$51: C6.1, R41.1
- new net N$52: IC5A.-IN, R41.2, R42.1
- new net N$53: C6.2, IC5A.OUT, R44.2
- new net N$54: IC5A.+IN, R43.1
- new net N$55: R39.1, R40.2, R43.2
- new net N$56: R39.2, R47.1
- new net N$57: IC6A.-IN, R48.1, R49.2
- new net N$58: IC6A.+IN, R50.1
- new net N$59: R50.2, R51.2, R52.1
- new net N$60: IC6A.OUT, IC7A.S2, R49.1
- new net N$61: IC7A.D, R42.2
- new net N$62: R53.1, R54.2
- new net N$63: R54.1, R55.2
- new net N$64: R55.1, R56.2
- new net N$65: R56.1, R57.2
- new net N$66: R57.1, R58.2, R60.2
- new net N$67: IC8A.OUT, R59.1, X1-18.F
- new net N$68: R61.2, R62.1, R63.2
- new net N$69: IC8A.+IN, R63.1
- new net N$70: IC8A.-IN, R59.2, R60.1
- new net N$71: R45.2, U$5G$2.S
- new net N$72: IC7A.S1, U$5G$4.S
- new net N$73: R46.2, U$5G$1.S
- new net N$74: OK2.A, R44.1
- net +15V: now also DC2.VIN+, IC5A.V+, IC6A.V+, IC7P.V+, IC8A.V+, R45.1, R52.2, R62.2
- net +5V: now also IC7VL.VL, U$7G$1.S
- net -15V: now also IC5A.V-, IC6A.V-, IC7P.V-, IC8A.V-, R46.1, R51.1, R61.1
- net GND: now also D13.A, DC2.VIN-, IC7P.GND, OK2.C, R40.1, R58.1, R64.1, U$6G$2.S
- net N$12: now also OK1.EMI; no longer OK1.EMIT
- net N$29: now also D8.C, D9.A; no longer IC3A.IN, R32.2, U$4G$2.S
- net V+: now also Q3.D, R37.2
- net V-: now also DC2.0V, R34.1, R38.1, T4.E
Other:
- moved on the sheet: C1, C2, C3, C4, C5, D1, D2, D3, D4, D5, D6, D7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
