File: eagle/regulator_plus_switch.sch (EAGLE design)
At the start: 60 parts, among them IC1 LT1352PA, IC2 LT1352PA, IC3 DG419DJN, IC4 LT1352PA, T1 2N3904, T2 2N3904

Commit message: pa 97 circuit
Parts:
- removed C5: 10n, rcl:C-US075-032X103
- removed D7: 1N4148DO35-10, diode:1N4148DO35-10
- removed DC1: (no value), dc-dc-converter:NCS
- removed IC1: LT1352PA, linear-technology:LT1352PA
- removed OK1: PC817, optocoupler:PC817
- removed Q1, Q2: (no value), transistor-power:PMOSFET_NTO220BV
- removed R1, R2: 65, rcl:R-US_0207/10
- removed R10, R11, R9: 10k, rcl:R-US_0207/10
- removed R12: 250, rcl:R-US_0207/15
- removed R15, R5, R7: 1M, resistor:R-US_0414/15
- removed R3, R4: 100, rcl:R-US_0207/10
- removed R6: 100k, rcl:R-US_0207/10
- removed R8: 50k, rcl:R-US_0207/10
- removed T1, T2: 2N3904, transistor:2N3904
- added U$3: PA97, apex:PA97
Connections:
- removed net N$11: Q2.G, R4.1
- removed net N$12: OK1.EMIT, R4.2, R6.2, T2.C
- removed net N$14: Q2.S, R2.2, T2.B
- removed net N$16: DC1.VOUT, OK1.COL
- removed net N$17: C5.1, R9.1
- removed net N$18: IC1A.-IN, R10.1, R9.2
- removed net N$19: C5.2, IC1A.OUT, R12.2
- removed net N$20: IC1A.+IN, R11.1
- removed net N$21: R11.2, R7.1, R8.2
- removed net N$22: OK1.A, R12.1
- removed net N$23: R15.1, R7.2
- removed net N$6: Q1.G, R3.1
- removed net N$7: D7.C, Q2.D, R3.2, R5.1, T1.C
- removed net N$8: Q1.S, R1.2, T1.B
- net +15V: no longer DC1.VIN+, IC1A.V+
- net -15V: no longer IC1A.V-
- net GND: no longer DC1.VIN-, OK1.C, R8.1
- net N$10: no longer D7.A, R1.1, R15.2, T1.E
- net N$28: no longer R10.2
- net V+: no longer Q1.D, R5.2
- net V-: no longer DC1.0V, R2.1, R6.1, T2.E
Other:
- moved on the sheet: U$2G$1, U$2G$2, U$2G$3, U$2G$4, X2-1, X2-2, X2-3, X2-4, X2-5, X2-6

Commit message: add display out
Parts:
- removed D4, D5: P6KEXX, diode:P6KEXX
- added J17: 5669-8, con-molex:5669-8
- added J23, J24, J25, J26: 5569-2, con-molex:5569-2
- added R1: 220, rcl:R-US_0207/10
- D1, D2, D3, D6: value P6KEXX -> P6KEXXA; device diode:P6KEXX -> diode:P6KEXXA
Connections:
- removed net N$2: D2.C, D3.A
- removed net N$3: D3.C, D4.C
- removed net N$4: D4.A, D5.C
- removed net N$5: D5.A, D6.C
- new net N$6: J23G$1.S, J24G$1.S
- new net N$7: J26G$1.S, R1.2
- net +5V: now also J25G$1.S, R1.1
- net GND: now also D2.A, D3.C, J23G$2.S, J24G$2.S, J25G$2.S, J26G$2.S
- net N$1: now also D6.C; no longer D2.A
- net N$34: now also J17G$1.S
- net V+: now also D2.C
- net V-: now also D3.A
Other:
- moved on the sheet: D1, D2, D3, D6
Changed lines of the file:
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@@
 </classes>
 <parts>
-<part name="D1" library="diode" deviceset="P6KEXX" device=""/>
-<part name="D2" library="diode" deviceset="P6KEXX" device=""/>
-<part name="D3" library="diode" deviceset="P6KEXX" device=""/>
-<part name="D4" library="diode" deviceset="P6KEXX" device=""/>
-<part name="D5" library="diode" deviceset="P6KEXX" device=""/>
-<part name="D6" library="diode" deviceset="P6KEXX" device=""/>
+<part name="D6" library="diode" deviceset="P6KEXXA" device=""/>
 <part name="FRAME1" library="frames" deviceset="FRAME_E_L" device=""/>
 <part name="C1" library="rcl" deviceset="C-US" device="075-032X103" value="10n"/>
@@
 <part name="U$5" library="con-amp-te" deviceset="640584-1" device=""/>
 <part name="U$3" library="apex" deviceset="PA97" device=""/>
+<part name="J17" library="con-molex" deviceset="5669-8" device=""/>
+<part name="J23" library="con-molex" deviceset="5569-2" device=""/>
+<part name="J24" library="con-molex" deviceset="5569-2" device=""/>
+<part name="J25" library="con-molex" deviceset="5569-2" device=""/>
+<part name="J26" library="con-molex" deviceset="5569-2" device=""/>
+<part name="P+3" library="supply1" deviceset="+5V" device=""/>
+<part name="GND5" library="supply1" deviceset="GND" device=""/>
+<part name="GND7" library="supply1" deviceset="GND" device=""/>
+<part name="GND8" library="supply1" deviceset="GND" device=""/>
+<part name="P+4" library="supply1" deviceset="+5V" device=""/>
+<part name="R1" library="rcl" deviceset="R-US_" device="0207/10" value="220"/>
+<part name="GND14" library="supply1" deviceset="GND" device=""/>
+<part name="D1" library="diode" deviceset="P6KEXXA" device=""/>
+<part name="P+5" library="supply1" deviceset="V+" device=""/>
+<part name="P-3" library="supply1" deviceset="V-" device=""/>
+<part name="D2" library="diode" deviceset="P6KEXXA" device=""/>
+<part name="D3" library="diode" deviceset="P6KEXXA" device=""/>
+<part name="GND26" library="supply1" deviceset="GND" device=""/>
+<part name="GND27" library="supply1" deviceset="GND" device=""/>
 </parts>
 <sheets>
@@
 </plain>
 <instances>
-<instance part="D1" gate="1" x="190.5" y="795.02" rot="R270"/>
-<instance part="D2" gate="1" x="190.5" y="789.94" rot="R270"/>
-<instance part="D3" gate="1" x="190.5" y="784.86" rot="R270"/>
-<instance part="D4" gate="1" x="190.5" y="779.78" rot="R90"/>
-<instance part="D5" gate="1" x="190.5" y="774.7" rot="R90"/>
-<instance part="D6" gate="1" x="190.5" y="769.62" rot="R90"/>
+<instance part="D6" gate="1" x="198.12" y="782.32" rot="R90"/>
 <instance part="FRAME1" gate="G$1" x="558.8" y="50.8"/>
 <instance part="C1" gate="G$1" x="241.3" y="815.34"/>
@@
 <instance part="C3" gate="G$1" x="264.16" y="815.34"/>
 <instance part="C4" gate="G$1" x="271.78" y="815.34"/>
-<instance part="GND6" gate="1" x="190.5" y="764.54"/>
+<instance part="GND6" gate="1" x="198.12" y="774.7"/>
 <instance part="P+7" gate="1" x="307.34" y="840.74" rot="R270"/>
 <instance part="P-6" gate="1" x="314.96" y="838.2" rot="R90"/>
@@
 <instance part="U$5" gate="G$8" x="205.74" y="746.76"/>
 <instance part="U$3" gate="G$1" x="91.44" y="797.56"/>
+<instance part="J17" gate="G$1" x="185.42" y="746.76"/>
+<instance part="J17" gate="G$2" x="187.96" y="693.42"/>
+<instance part="J17" gate="G$3" x="187.96" y="690.88"/>
+<instance part="J17" gate="G$4" x="187.96" y="688.34"/>
+<instance part="J17" gate="G$5" x="187.96" y="683.26"/>
+<instance part="J17" gate="G$6" x="187.96" y="680.72"/>
+<instance part="J17" gate="G$7" x="187.96" y="678.18"/>
+<instance part="J17" gate="G$8" x="187.96" y="675.64"/>
+<instance part="J23" gate="G$1" x="213.36" y="843.28"/>
+<instance part="J23" gate="G$2" x="236.22" y="843.28"/>
+<instance part="J24" gate="G$1" x="213.36" y="840.74"/>
+<instance part="J24" gate="G$2" x="236.22" y="838.2"/>
+<instance part="J25" gate="G$1" x="213.36" y="817.88"/>
+<instance part="J25" gate="G$2" x="213.36" y="815.34"/>
+<instance part="J26" gate="G$1" x="213.36" y="810.26"/>
+<instance part="J26" gate="G$2" x="213.36" y="807.72"/>
+<instance part="P+3" gate="1" x="208.28" y="817.88" rot="R90"/>
+<instance part="GND5" gate="1" x="208.28" y="815.34" rot="R270"/>
+<instance part="GND7" gate="1" x="231.14" y="843.28" rot="R270"/>
+<instance part="GND8" gate="1" x="231.14" y="838.2" rot="R270"/>
+<instance part="P+4" gate="1" x="193.04" y="810.26" rot="R90"/>
+<instance part="R1" gate="G$1" x="203.2" y="810.26"/>
+<instance part="GND14" gate="1" x="208.28" y="807.72" rot="R270"/>
+<instance part="D1" gate="1" x="198.12" y="795.02" rot="R270"/>
+<instance part="P+5" gate="1" x="264.16" y="840.74"/>
+<instance part="P-3" gate="1" x="271.78" y="840.74" rot="R180"/>
+<instance part="D2" gate="1" x="264.16" y="830.58" rot="R90"/>
+<instance part="D3" gate="1" x="271.78" y="835.66" rot="R270"/>
+<instance part="GND26" gate="1" x="264.16" y="825.5"/>
+<instance part="GND27" gate="1" x="271.78" y="825.5"/>
 </instances>
 <busses>
 </busses>
 <nets>
-<net name="N$1" class="0">
-<segment>
-<pinref part="D1" gate="1" pin="C"/>
-<pinref part="D2" gate="1" pin="A"/>
-</segment>
-</net>
-<net name="N$2" class="0">
-<segment>
-<pinref part="D2" gate="1" pin="C"/>
-<pinref part="D3" gate="1" pin="A"/>
-</segment>
-</net>
-<net name="N$3" class="0">
-<segment>
-<pinref part="D3" gate="1" pin="C"/>
-<pinref part="D4" gate="1" pin="C"/>
-</segment>
-</net>
-<net name="N$4" class="0">
-<segment>
-<pinref part="D4" gate="1" pin="A"/>
-<pinref part="D5" gate="1" pin="C"/>
-</segment>
-</net>
-<net name="N$5" class="0">
-<segment>
-<pinref part="D5" gate="1" pin="A"/>
-<pinref part="D6" gate="1" pin="C"/>
-</segment>
-</net>
 <net name="GND" class="0">
 <segment>
@@
 <pinref part="D6" gate="1" pin="A"/>
 <pinref part="GND6" gate="1" pin="GND"/>
+<wire x1="198.12" y1="779.78" x2="198.12" y2="777.24" width="0.1524" layer="91"/>
 </segment>
 <segment>
@@
 <pinref part="GND25" gate="1" pin="GND"/>
 </segment>
+<segment>
+<pinref part="J25" gate="G$2" pin="S"/>
+<pinref part="GND5" gate="1" pin="GND"/>
+</segment>
+<segment>
+<pinref part="J23" gate="G$2" pin="S"/>
+<pinref part="GND7" gate="1" pin="GND"/>
+</segment>
+<segment>
+<pinref part="J24" gate="G$2" pin="S"/>
+<pinref part="GND8" gate="1" pin="GND"/>
+</segment>
+<segment>
+<pinref part="J26" gate="G$2" pin="S"/>
+<pinref part="GND14" gate="1" pin="GND"/>
+</segment>
+<segment>
+<pinref part="D2" gate="1" pin="A"/>
+<pinref part="GND26" gate="1" pin="GND"/>
+</segment>
+<segment>
+<pinref part="D3" gate="1" pin="C"/>
+<pinref part="GND27" gate="1" pin="GND"/>
+<wire x1="271.78" y1="828.04" x2="271.78" y2="833.12" width="0.1524" layer="91"/>
+</segment>
 </net>
 <net name="V+" class="0">
@@
 <wire x1="304.8" y1="840.74" x2="297.18" y2="840.74" width="0.1524" layer="91"/>
 </segment>
+<segment>
+<pinref part="P+5" gate="1" pin="V+"/>
+<pinref part="D2" gate="1" pin="C"/>
+<wire x1="264.16" y1="833.12" x2="264.16" y2="838.2" width="0.1524" layer="91"/>
+</segment>
 </net>
 <net name="V-" class="0">
@@
 <wire x1="312.42" y1="838.2" x2="297.18" y2="838.2" width="0.1524" layer="91"/>
 </segment>
+<segment>
+<pinref part="P-3" gate="1" pin="V-"/>
+<pinref part="D3" gate="1" pin="A"/>
+</segment>
 </net>
 <net name="N$10" class="0">
 <segment>
+<pinref part="R21" gate="G$1" pin="2"/>
+<wire x1="203.2" y1="797.56" x2="198.12" y2="797.56" width="0.1524" layer="91"/>
+<pinref part="U$5" gate="G$1" pin="P$1"/>
 <pinref part="D1" gate="1" pin="A"/>
-<wire x1="182.88" y1="797.56" x2="190.5" y2="797.56" width="0.1524" layer="91"/>
-<pinref part="R21" gate="G$1" pin="2"/>
-<wire x1="203.2" y1="797.56" x2="190.5" y2="797.56" width="0.1524" layer="91"/>
-<pinref part="U$5" gate="G$1" pin="P$1"/>
+<wire x1="198.12" y1="797.56" x2="182.88" y2="797.56" width="0.1524" layer="91"/>
+<junction x="198.12" y="797.56"/>
 </segment>
 </net>
@@
 <pinref part="P+18" gate="1" pin="+5V"/>
 <wire x1="58.42" y1="695.96" x2="63.5" y2="695.96" width="0.1524" layer="91"/>
+</segment>
+<segment>
+<pinref part="J25" gate="G$1" pin="S"/>
+<pinref part="P+3" gate="1" pin="+5V"/>
+</segment>
+<segment>
+<pinref part="P+4" gate="1" pin="+5V"/>
+<pinref part="R1" gate="G$1" pin="1"/>
+<wire x1="195.58" y1="810.26" x2="198.12" y2="810.26" width="0.1524" layer="91"/>
 </segment>
 </net>
@@
 <wire x1="172.72" y1="726.44" x2="119.38" y2="726.44" width="0.1524" layer="91"/>
 <wire x1="119.38" y1="726.44" x2="119.38" y2="751.84" width="0.1524" layer="91"/>
+<pinref part="J17" gate="G$1" pin="S"/>
+<junction x="182.88" y="746.76"/>
 </segment>
 </net>
@@
 </segment>
 </net>
+<net name="N$6" class="0">
+<segment>
+<pinref part="J23" gate="G$1" pin="S"/>
+<pinref part="J24" gate="G$1" pin="S"/>
+<wire x1="210.82" y1="843.28" x2="210.82" y2="840.74" width="0.1524" layer="91"/>
+</segment>
+</net>
+<net name="N$7" class="0">
+<segment>
+<pinref part="J26" gate="G$1" pin="S"/>
+<pinref part="R1" gate="G$1" pin="2"/>
+<wire x1="208.28" y1="810.26" x2="210.82" y2="810.26" width="0.1524" layer="91"/>
+</segment>
+</net>
+<net name="N$1" class="0">
+<segment>
+<pinref part="D6" gate="1" pin="C"/>
+<pinref part="D1" gate="1" pin="C"/>
+<wire x1="198.12" y1="792.48" x2="198.12" y2="784.86" width="0.1524" layer="91"/>
+</segment>
+</net>

Commit message: Test layouts pa97
Parts:
- removed D1, D6: P6KEXXA, diode:P6KEXXA
- removed J17: 5669-8, con-molex:5669-8
- removed U$3: PA97, apex:PA97
- removed U$5: 640584-1, con-amp-te:640584-1
- added C5, C7: 10p, rcl:C-US075-032X103
- added C6: 10n, rcl:C-US075-032X103
- added D10, D9: 1n4742, diode:ZENER-DIODEDO41Z10
- added D7, D8: P6KEXXA, diode:P6KEXXA
- added DISPLAY: 5669-8, con-molex:5669-8
- added KK1: SK125/50C247, heatsink:SK125/50C247
- added MAN/EXT: 5569-2, con-molex:5569-2
- added OUT: 640584-1, con-amp-te:640584-1
- added R2, R3, R4: 1M, rcl:R-US_0207/10
- added R5, R6, R7: 25.5k, rcl:R-US_0207/10
- R21, R22, R23, R24, R25: device resistor:R-US_0414/15 -> resistor:R-US_0207/10
- R26: value 50k -> 5k
- R32: device rcl:R-US_0207/10 -> rcl:R-US_0207/15
- U$4: value 5569-2 -> PA97; device con-molex:5569-2 -> apex:PA97
- renumbered J23 to UNK, J24 to GROUND, J25 to DISPLAYPOWER, J26 to LED, U$1 to POT1, U$2 to HVIN, X1 to EXTERNAL, X2 to POWER
Connections:
- removed net N$1: D1.C, D6.C
- removed net N$10: D1.A, R21.2, U$5G$1.P$1
- new net N$11: C7.2, D8.A, OUTG$1.P$1, R21.2, R3.2, U$4.OUT
- new net N$12: R2.1, R4.2
- new net N$14: R5.1, R6.2
- new net N$16: R6.1, R7.1
- new net N$18: R2.2, R3.1
- new net N$29: D10.C, D9.C
- new net N$3: C5.1, U$4.CC1
- new net N$38: C7.1, D10.A, R4.1, R5.2, U$4.-IN
- new net N$4: C5.2, U$4.CC2
- new net N$8: D7.C, D8.C
- net +5V: now also C6.1, MAN/EXTG$1.S; no longer U$4G$1.S
- net GND: now also C6.2, D7.A, R7.2; no longer D6.A
- net MAN: now also MAN/EXTG$2.S; no longer U$4G$2.S
- net N$28: now also D9.A, U$4.+IN
- net N$34: now also DISPLAYG$1.S; no longer J17G$1.S
- net V+: now also U$4.V+
- net V-: now also U$4.V-
Other:
- moved on the sheet: R21, R22, R23, R24, R25, R26

Commit message: regulator
Parts:
- added C8, C9: cc, rcl:C-US075-032X103
- added Q1, Q2: 2N3906, transistor-pnp:2N3906
- added R10, R12: rb, rcl:R-US_0207/10
- added R11, R8: rlim, rcl:R-US_0207/10
- added R15, R9: rl, rcl:R-US_0207/10
- added T1, T2: 2N3904, transistor:2N3904
Connections:
- net N$28 renamed VIN+
- net N$38 renamed VIN-
- new net N$1: R11.2, R12.2, T2.E
- new net N$10: C8.2, Q1.B, Q2.C, R9.2
- new net N$17: C9.2, R12.1, T1.B
- new net N$19: C9.1, R15.1, T1.C, T2.B
- new net N$2: C8.1, Q2.B, R10.1
- new net N$5: Q1.E, R10.2, R8.1
- new net V+_SAFE: Q1.C, U$4.V+
- new net V-_SAFE: T2.C, U$4.V-
- net GND: now also R15.2, R9.1
- net V+: now also Q2.E, R8.2; no longer U$4.V+
- net V-: now also R11.1, T1.E; no longer U$4.V-
Other:
- moved on the sheet: KK1
