File: eagle/test_ckt.sch (EAGLE design)
At the start: 38 parts, among them IC1 LT1352PA, T1 2N3904, T2 2N3904

Commit message: "Works" but not full scale yet
Parts:
- OK1: value CNY17 -> PC817; device optocoupler:CNY17 -> optocoupler:PC817
Connections:
- net N$12: now also OK1.EMIT; no longer OK1.EMI
Changed lines of the file:
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@@
 <part name="P-8" library="supply1" deviceset="-15V" device=""/>
 <part name="P+6" library="supply1" deviceset="+15V" device=""/>
-<part name="OK1" library="optocoupler" deviceset="CNY17" device=""/>
+<part name="OK1" library="optocoupler" deviceset="PC817" device=""/>
 </parts>
 <sheets>
@@
 <instance part="P-8" gate="1" x="190.5" y="142.24" rot="R180"/>
 <instance part="P+6" gate="1" x="114.3" y="154.94"/>
-<instance part="OK1" gate="G$1" x="106.68" y="111.76"/>
+<instance part="OK1" gate="A" x="106.68" y="109.22"/>
 </instances>
 <busses>
@@
 <segment>
 <pinref part="GND8" gate="1" pin="GND"/>
-<pinref part="OK1" gate="G$1" pin="C"/>
+<pinref part="OK1" gate="A" pin="C"/>
 </segment>
 </net>
@@
 <pinref part="R6" gate="G$1" pin="2"/>
 <wire x1="119.38" y1="106.68" x2="114.3" y2="106.68" width="0.1524" layer="91"/>
-<pinref part="OK1" gate="G$1" pin="EMI"/>
+<pinref part="OK1" gate="A" pin="EMIT"/>
 <junction x="114.3" y="106.68"/>
 </segment>
@@
 <pinref part="DC1" gate="G$1" pin="VOUT"/>
 <wire x1="114.3" y1="121.92" x2="114.3" y2="116.84" width="0.1524" layer="91"/>
-<pinref part="OK1" gate="G$1" pin="COL"/>
 <wire x1="114.3" y1="111.76" x2="116.84" y2="111.76" width="0.1524" layer="91"/>
 <wire x1="116.84" y1="111.76" x2="116.84" y2="116.84" width="0.1524" layer="91"/>
 <wire x1="116.84" y1="116.84" x2="114.3" y2="116.84" width="0.1524" layer="91"/>
+<pinref part="OK1" gate="A" pin="COL"/>
 </segment>
 </net>
@@
 <net name="N$25" class="0">
 <segment>
-<pinref part="OK1" gate="G$1" pin="A"/>
 <pinref part="R12" gate="G$1" pin="1"/>
 <wire x1="96.52" y1="114.3" x2="96.52" y2="111.76" width="0.1524" layer="91"/>
-</segment>
-</net>
+<pinref part="OK1" gate="A" pin="A"/>
+<junction x="96.52" y="111.76"/>
+</segment>
+</net>
