File: eagle/test_ckt.brd (EAGLE design)
At the start: 152.4 x 152.4 mm, 38 parts, among them IC1 LT1352PA, T1 2N3904, T2 2N3904

Commit message: "Works" but not full scale yet
Parts:
- OK1: value CNY17 -> PC817; device optocoupler:DIL06 -> optocoupler:DIL04
- moved OK1 0.80 mm to (62.5, 74.2)
Connections:
- net N$12: now also OK1.3; no longer OK1.4
- net N$16: now also OK1.4; no longer OK1.5
Routing:
- net N$8: track 14.5 -> 23.4 mm
- net N$25: track 30.3 -> 29.7 mm
- added copper zone on layer 1, net GND
Other:
- board size 152.4 x 152.4 mm -> 152.4 x 132.1 mm
Changed lines of the file:
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@@
 <plain>
 <wire x1="0" y1="0" x2="152.4" y2="0" width="0" layer="20"/>
-<wire x1="152.4" y1="0" x2="152.4" y2="152.4" width="0" layer="20"/>
-<wire x1="152.4" y1="152.4" x2="0" y2="152.4" width="0" layer="20"/>
-<wire x1="0" y1="152.4" x2="0" y2="0" width="0" layer="20"/>
-<text x="63.246" y="83.82" size="1.778" layer="51">2n3904 are on reverse side!!!</text>
-<text x="9.144" y="141.986" size="1.778" layer="51">2n3904 are on reverse side!!!</text>
-<text x="53.848" y="138.684" size="1.778" layer="51">2n3904 are on reverse side!!!</text>
-<text x="71.374" y="145.034" size="1.778" layer="51">2n3904 are on reverse side!!!</text>
-<text x="92.456" y="135.89" size="1.778" layer="51">2n3904 are on reverse side!!!</text>
-<text x="107.188" y="143.51" size="1.778" layer="51">2n3904 are on reverse side!!!</text>
-<text x="5.588" y="132.334" size="1.778" layer="51">2n3904 are on reverse side!!!</text>
-<text x="61.468" y="131.826" size="1.778" layer="51">2n3904 are on reverse side!!!</text>
+<wire x1="152.4" y1="0" x2="152.4" y2="132.08" width="0" layer="20"/>
+<wire x1="152.4" y1="132.08" x2="0" y2="132.08" width="0" layer="20"/>
+<wire x1="0" y1="132.08" x2="0" y2="0" width="0" layer="20"/>
+<text x="76.2" y="49.276" size="1.778" layer="51">2n3904 are on reverse side!!!</text>
+<text x="63.754" y="83.058" size="1.778" layer="51">2n3904 are on reverse side!!!</text>
 </plain>
 <attributes>
@@
 <element name="R13" library="rcl" package="0207/10" value="20k" x="9.144" y="32.766"/>
 <element name="R14" library="rcl" package="0207/10" value="20k" x="31.242" y="35.814" rot="R180"/>
-<element name="OK1" library="optocoupler" package="DIL06" value="CNY17" x="62.23" y="74.93" rot="R270">
-<attribute name="OC_NEWARK" value="05M4044" x="62.23" y="74.93" size="1.778" layer="27" rot="R270" display="off"/>
-<attribute name="MPN" value="CNY17-1" x="62.23" y="74.93" size="1.778" layer="27" rot="R270" display="off"/>
-<attribute name="MF" value="" x="62.23" y="74.93" size="1.778" layer="27" rot="R270" display="off"/>
-<attribute name="OC_FARNELL" value="1045399" x="62.23" y="74.93" size="1.778" layer="27" rot="R270" display="off"/>
+<element name="OK1" library="optocoupler" package="DIL04" value="PC817" x="62.484" y="74.168" rot="R270">
+<attribute name="OC_NEWARK" value="97K7059" x="62.484" y="74.168" size="1.778" layer="27" rot="R270" display="off"/>
+<attribute name="MPN" value="PC817X4J000F" x="62.484" y="74.168" size="1.778" layer="27" rot="R270" display="off"/>
+<attribute name="MF" value="" x="62.484" y="74.168" size="1.778" layer="27" rot="R270" display="off"/>
+<attribute name="OC_FARNELL" value="9707727" x="62.484" y="74.168" size="1.778" layer="27" rot="R270" display="off"/>
 </element>
 </elements>
@@
 <vertex x="0" y="0"/>
 <vertex x="152.4" y="0"/>
-<vertex x="152.4" y="152.4"/>
-<vertex x="0" y="152.4"/>
+<vertex x="152.146" y="132.334"/>
+<vertex x="-0.762" y="132.08"/>
 </polygon>
 <contactref element="U$3" pad="P$2"/>
@@
 <contactref element="X1" pad="3"/>
 <contactref element="OK1" pad="2"/>
+<polygon width="0.4064" layer="1" isolate="1.4224" thermals="no">
+<vertex x="-0.508" y="131.826"/>
+<vertex x="152.146" y="132.334"/>
+<vertex x="152.4" y="-0.254"/>
+<vertex x="0" y="-0.254"/>
+</polygon>
 </signal>
 <signal name="V+">
@@
 <wire x1="100.965" y1="96.52" x2="102.87" y2="96.52" width="1.4224" layer="16"/>
 <wire x1="102.87" y1="96.52" x2="111.76" y2="105.41" width="1.4224" layer="16"/>
-<wire x1="111.76" y1="105.41" x2="111.76" y2="114.3" width="0" layer="19" extent="1-1"/>
+<wire x1="111.76" y1="114.3" x2="111.76" y2="105.41" width="1.4224" layer="16"/>
 </signal>
 <signal name="N$10">
@@
 <contactref element="R6" pad="2"/>
 <wire x1="76.2" y1="78.74" x2="76.2" y2="72.136" width="1.4224" layer="16"/>
-<wire x1="76.2" y1="72.136" x2="76.2" y2="69.85" width="1.4224" layer="16"/>
+<wire x1="76.2" y1="72.136" x2="76.2" y2="71.882" width="1.4224" layer="16"/>
+<wire x1="76.2" y1="71.882" x2="76.2" y2="69.85" width="1.4224" layer="16"/>
 <wire x1="87.63" y1="64.77" x2="82.55" y2="69.85" width="1.4224" layer="16"/>
 <wire x1="82.55" y1="69.85" x2="76.2" y2="69.85" width="1.4224" layer="16"/>
-<contactref element="OK1" pad="4"/>
-<wire x1="66.04" y1="72.39" x2="75.946" y2="72.39" width="1.4224" layer="16"/>
 <wire x1="75.946" y1="72.39" x2="76.2" y2="72.136" width="1.4224" layer="16"/>
 <wire x1="87.63" y1="64.77" x2="87.63" y2="62.23" width="1.4224" layer="16"/>
+<contactref element="OK1" pad="3"/>
+<wire x1="66.294" y1="72.898" x2="75.184" y2="72.898" width="1.4224" layer="16"/>
+<wire x1="75.184" y1="72.898" x2="76.2" y2="71.882" width="1.4224" layer="16"/>
 </signal>
 <signal name="N$14">
@@
 <wire x1="63.754" y1="65.786" x2="66.04" y2="63.5" width="1.4224" layer="16"/>
 <wire x1="66.04" y1="63.5" x2="66.04" y2="59.69" width="1.4224" layer="16"/>
-<contactref element="OK1" pad="5"/>
-<wire x1="66.04" y1="74.93" x2="63.754" y2="74.93" width="1.4224" layer="16"/>
 <wire x1="63.754" y1="74.93" x2="63.754" y2="65.786" width="1.4224" layer="16"/>
+<contactref element="OK1" pad="4"/>
+<wire x1="66.294" y1="75.438" x2="64.262" y2="75.438" width="1.4224" layer="16"/>
+<wire x1="64.262" y1="75.438" x2="63.754" y2="74.93" width="1.4224" layer="16"/>
 </signal>
 <signal name="N$17">
@@
 </signal>
 <signal name="N$25">
-<contactref element="OK1" pad="1"/>
 <contactref element="R12" pad="1"/>
 <wire x1="29.21" y1="74.93" x2="48.768" y2="74.93" width="1.4224" layer="16"/>
-<wire x1="48.768" y1="74.93" x2="51.308" y2="77.47" width="1.4224" layer="16"/>
-<wire x1="51.308" y1="77.47" x2="58.42" y2="77.47" width="1.4224" layer="16"/>
+<wire x1="48.768" y1="74.93" x2="49.276" y2="75.438" width="1.4224" layer="16"/>
+<contactref element="OK1" pad="1"/>
+<wire x1="58.674" y1="75.438" x2="49.276" y2="75.438" width="1.4224" layer="16"/>
 </signal>
 </signals>

Commit message: pa 97 circuit
Parts:
- removed T2: 2N3904, transistor:TO92
- added Q3, Q4: C2M0280120D90H, transistor-power:TO-247AD-V
- R12: value 250 -> 20k
- R2: value 65 -> 5k
- R6: value 100k -> 10k
- moved R11 9.40 mm to (70.4, 36.8)
- moved R10 7.88 mm to (61.2, 30.7)
- moved R6 4.02 mm to (74.9, 68.6), turned to 270 degrees
- moved R4 3.34 mm to (81.8, 75.4)
- moved Q2 3.30 mm to (96.5, 78.0)
- moved OK1 1.52 mm to (61.0, 74.2)
Connections:
- removed net N$20: IC1.3, R11.1
- new net N$22: OK1.4, R4.2, R6.1
- net -15V: now also OK1.2
- net GND: no longer OK1.2
- net N$12: now also IC1.3, R10.1; no longer OK1.3, R4.2, R6.2, T2.1
- net N$14: no longer T2.2
- net N$16: now also R6.2; no longer OK1.4
- net N$18: now also R11.1; no longer R10.1
- net V-: now also OK1.3; no longer R6.1, T2.3
Routing:
- net N$12: track 35.7 -> 10.2 mm
- net N$18: track 17.8 -> 37.4 mm
- net N$20: track 15.5 -> 0.00 mm
- net N$14: track 24.3 -> 9.40 mm
- net N$22: track 0.00 -> 13.7 mm
- net -15V: track 108.3 -> 119.7 mm
- net N$21: track 54.6 -> 45.2 mm
- net N$13: track 75.3 -> 83.0 mm
- net N$16: track 18.9 -> 12.7 mm
- net V-: track 139.7 -> 135.9 mm
- net N$7: track 81.3 -> 84.6 mm
- net N$25: track 29.7 -> 28.2 mm
- net N$11: track 7.62 -> 7.11 mm
- removed copper zone on layer 1, net GND
Other:
- board size 152.4 x 132.1 mm -> 152.4 x 152.4 mm
