File: eagle/test_ckt_2.brd (EAGLE design)
At the start: 184.7 x 181.9 mm, 60 parts, among them IC1 LT1352PA, IC2 LT1352PA, IC3 DG419DJN, IC4 LT1352PA, T1 2N3904, T2 2N3904

Commit message: Solution to full scale?
Parts:
- removed IC2, IC4: LT1352PA, linear-technology:DIL08
- removed IC3: DG419DJN, linear:DIL08
- removed R16, R18, R27, R31: 10k, rcl:0207/10
- removed R17, R28: 40k, rcl:0207/10
- removed R19, R29: 17k, rcl:0207/10
- removed R20, R30: 13k, rcl:0207/10
- removed R21, R22, R23, R24, R25: 1M, resistor:0414/15
- removed R26: 50k, rcl:0207/10
- removed R32: 100k, rcl:0207/10
- removed T1, T2: 2N3904, transistor:TO92
- removed U$4: 5569-2, con-molex:5569-2
- removed U$5: 640584-1, con-amp-te:640584-1
- removed X2: (no value), con-molex:KK-156-6
- added D8: (no value), diode:ZDIO12.5
- added U$3: 5569-2, con-molex:5569-2
- D7: value 1N4148DO35-10 -> (none); device diode:DO35-10 -> diode:ZDIO12.5
- R1: value 65 -> 25k
- R12: value 250 -> 25k
- R13, R14: device rcl:0207/15 -> rcl:0207/10
- R2: value 65 -> 2k
- R6: value 100k -> 25k
- X1: device con-subd:F25HP -> con-molex:KK-156-6
- moved X1 165.7 mm to (6.35, 53.3)
- moved C1 81.5 mm to (15.2, 47.2)
- moved U$1 61.7 mm to (14.0, 17.3)
- moved R14 54.6 mm to (31.2, 35.8)
- moved D2 52.5 mm to (137.2, 91.4)
- moved D4 52.5 mm to (137.2, 61.0)
- moved D3 52.5 mm to (127.0, 76.2)
- moved D5 52.5 mm to (127.0, 45.7)
- moved D6 52.5 mm to (137.2, 30.5)
- moved D1 52.5 mm to (127.0, 106.7)
- moved C5 52.5 mm to (33.3, 15.2)
- moved Q2 52.3 mm to (96.5, 81.3)
- moved R15 52.3 mm to (111.8, 77.5)
- moved R2 52.3 mm to (99.1, 61.0)
- moved C2 52.3 mm to (19.1, 72.4)
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Connections:
- removed net CMD1: R16.2, X1.1
- removed net MAN: IC3.6, R32.2, U$4.P$2
- removed net N$24 (its old number): IC2.2, R16.1, R17.2
- removed net N$25 (its old number): IC2.3, R18.1
- removed net N$26: R18.2, R19.2, R20.1
- removed net N$27: IC2.1, IC3.8, R17.1
- removed net N$28: IC3.1, R10.2
- removed net N$30: R21.1, R22.2
- removed net N$31: R22.1, R23.2
- removed net N$32: R23.1, R24.2
- removed net N$33: R24.1, R25.2
- removed net N$34: R25.1, R26.2, R28.2
- removed net N$35: IC4.1, R27.1, X1.17
- removed net N$36: R29.2, R30.1, R31.2
- removed net N$37: IC4.3, R31.1
- removed net N$39: IC4.2, R27.2, R28.1
- net +15V: now also C1.1, X1.6; no longer C2.1, IC2.8, IC3.4, IC4.8, R20.2, R30.2, X2.6
- net +5V: now also X1.4, X1.5; no longer IC3.5, U$4.P$1, X2.4, X2.5
- net -15V: now also C2.1, X1.1; no longer C1.1, IC2.4, IC3.7, IC4.4, R19.1, R29.1, X2.1
- net GND: now also U$3.P$2, X1.3; no longer IC3.3, R26.1, R32.1, X1.10, X1.12, X1.14, X1.16, X1.25, X1.4, X1.6, X1.8, X2.2, X2.3
- net N$10: now also U$3.P$1; no longer R21.2, T1.3, U$5.P$1
- net N$12: now also D8.C; no longer T2.1
- net N$13: now also R10.2; no longer IC3.2
- net N$14: no longer T2.2
- net N$7: no longer T1.1
- net N$8: no longer T1.2
- net V-: now also D8.A; no longer T2.3
Routing:
- net N$35: track 212.7 -> 0.00 mm
- net CMD1: track 131.9 -> 0.00 mm
- net +15V: track 235.6 -> 107.9 mm, vias 4 -> 0
- net -15V: track 232.2 -> 108.3 mm, vias 2 -> 0
- net +5V: track 115.3 -> 0.00 mm
- net N$34: track 85.2 -> 0.00 mm
- net MAN: track 56.6 -> 0.00 mm
- net GND: track 51.3 -> 2.54 mm, vias 4 -> 0
- net N$39: track 31.6 -> 0.00 mm
- net N$10: track 115.7 -> 85.9 mm
- net N$36: track 29.0 -> 0.00 mm
- net N$18: track 42.0 -> 17.8 mm
- net N$24 (its old number): track 23.4 -> 0.00 mm
- net N$26: track 22.9 -> 0.00 mm
- net N$14: track 41.6 -> 19.9 mm, vias 2 -> 0
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- added copper zone on layer 1, net GND
Other:
- board size 184.7 x 181.9 mm -> 152.4 x 132.1 mm
- board text added: "2n3904 are on reverse side!!!"

Commit message: pa 97 circuit
Parts:
- removed D8: (no value), diode:ZDIO12.5
Connections:
- net N$12: no longer D8.C
- net V-: no longer D8.A
Changed lines of the file:
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@@
 <attribute name="OC_FARNELL" value="9707727" x="62.484" y="74.168" size="1.778" layer="27" rot="R270" display="off"/>
 </element>
-<element name="D8" library="diode" package="ZDIO12.5" value="" x="7.62" y="-4.064"/>
 </elements>
 <signals>
@@
 <wire x1="20.7518" y1="116.84" x2="20.7518" y2="104.9782" width="1.4224" layer="16"/>
 <wire x1="20.7518" y1="104.9782" x2="30.48" y2="95.25" width="1.4224" layer="16"/>
-<contactref element="D8" pad="A"/>
-<wire x1="13.843" y1="-4.064" x2="63.5" y2="55.88" width="0" layer="19" extent="16-16"/>
 </signal>
 <signal name="N$6">
@@
 <wire x1="66.294" y1="72.898" x2="75.184" y2="72.898" width="1.4224" layer="16"/>
 <wire x1="75.184" y1="72.898" x2="76.2" y2="71.882" width="1.4224" layer="16"/>
-<contactref element="D8" pad="C"/>
-<wire x1="1.27" y1="-4.064" x2="66.294" y2="72.898" width="0" layer="19" extent="1-1"/>
 </signal>
 <signal name="N$14">
