File: eagle/test_ckt_2.sch (EAGLE design)
At the start: 60 parts, among them IC1 LT1352PA, IC2 LT1352PA, IC3 DG419DJN, IC4 LT1352PA, T1 2N3904, T2 2N3904

Commit message: Solution to full scale?
Parts:
- removed IC2, IC4: LT1352PA, linear-technology:LT1352PA
- removed IC3: DG419DJN, linear:DG419DJN
- removed R16, R18, R27, R31: 10k, rcl:R-US_0207/10
- removed R17, R28: 40k, rcl:R-US_0207/10
- removed R19, R29: 17k, rcl:R-US_0207/10
- removed R20, R30: 13k, rcl:R-US_0207/10
- removed R21, R22, R23, R24, R25: 1M, resistor:R-US_0414/15
- removed R26: 50k, rcl:R-US_0207/10
- removed R32: 100k, rcl:R-US_0207/10
- removed T1, T2: 2N3904, transistor:2N3904
- removed U$4: 5569-2, con-molex:5569-2
- removed U$5: 640584-1, con-amp-te:640584-1
- removed X2: (no value), con-molex:KK-156-6
- added D8: (no value), diode:ZENER-DIODEZD-12.5
- added U$3: 5569-2, con-molex:5569-2
- D7: value 1N4148DO35-10 -> (none); device diode:1N4148DO35-10 -> diode:ZENER-DIODEZD-12.5
- R1: value 65 -> 25k
- R12: value 250 -> 25k
- R13, R14: device rcl:R-US_0207/15 -> rcl:R-US_0207/10
- R2: value 65 -> 2k
- R6: value 100k -> 25k
- X1: device con-subd:F25HPS -> con-molex:KK-156-6
Connections:
- removed net CMD1: R16.2, X1-1.F
- removed net MAN: IC3A.IN, R32.2, U$4G$2.S
- removed net N$24 (its old number): IC2A.-IN, R16.1, R17.2
- removed net N$25 (its old number): IC2A.+IN, R18.1
- removed net N$26: R18.2, R19.2, R20.1
- removed net N$27: IC2A.OUT, IC3A.S2, R17.1
- removed net N$28: IC3A.D, R10.2
- removed net N$30: R21.1, R22.2
- removed net N$31: R22.1, R23.2
- removed net N$32: R23.1, R24.2
- removed net N$33: R24.1, R25.2
- removed net N$34: R25.1, R26.2, R28.2
- removed net N$35: IC4A.OUT, R27.1, X1-17.F
- removed net N$36: R29.2, R30.1, R31.2
- removed net N$37: IC4A.+IN, R31.1
- removed net N$39: IC4A.-IN, R27.2, R28.1
- net +15V: now also C1.1, X1-6.S; no longer C2.1, IC2A.V+, IC3P.V+, IC4A.V+, R20.2, R30.2, X2-6.S
- net +5V: now also X1-4.S, X1-5.S; no longer IC3VL.VL, U$4G$1.S, X2-4.S, X2-5.S
- net -15V: now also C2.1, X1-1.S; no longer C1.1, IC2A.V-, IC3P.V-, IC4A.V-, R19.1, R29.1, X2-1.S
- net GND: now also U$3G$2.S, X1-2.S, X1-3.S; no longer IC3P.GND, R26.1, R32.1, X1-10.F, X1-12.F, X1-14.F, X1-16.F, X1-2.F, X1-25.F, X1-4.F, X1-6.F, X1-8.F, X2-2.S, X2-3.S
- net N$10: now also U$3G$1.S; no longer R21.2, T1.E, U$5G$1.P$1
- net N$12: now also D8.C; no longer T2.C
- net N$13: now also R10.2; no longer IC3A.S1
- net N$14: no longer T2.B
- net N$7: no longer T1.C
- net N$8: no longer T1.B
- net V-: now also D8.A; no longer T2.E
Other:
- moved on the sheet: C1, C2, C3, C4, C5, D1, D2, D3, D4, D5, D6, IC1A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

Commit message: pa 97 circuit
Parts:
- removed D8: (no value), diode:ZENER-DIODEZD-12.5
Connections:
- net N$12: no longer D8.C
- net V-: no longer D8.A
Changed lines of the file:
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@@
 <part name="P+6" library="supply1" deviceset="+15V" device=""/>
 <part name="OK1" library="optocoupler" deviceset="PC817" device=""/>
-<part name="D8" library="diode" deviceset="ZENER-DIODE" device="ZD-12.5"/>
 </parts>
 <sheets>
@@
 <instance part="P+6" gate="1" x="114.3" y="154.94"/>
 <instance part="OK1" gate="A" x="106.68" y="109.22"/>
-<instance part="D8" gate="G$1" x="119.38" y="104.14" rot="R90"/>
 </instances>
 <busses>
@@
 <segment>
 <pinref part="R2" gate="G$1" pin="1"/>
-<wire x1="134.62" y1="91.44" x2="119.38" y2="91.44" width="0.1524" layer="91"/>
+<wire x1="134.62" y1="91.44" x2="114.3" y2="91.44" width="0.1524" layer="91"/>
 <pinref part="R6" gate="G$1" pin="1"/>
-<wire x1="119.38" y1="91.44" x2="114.3" y2="91.44" width="0.1524" layer="91"/>
 <wire x1="114.3" y1="91.44" x2="114.3" y2="96.52" width="0.1524" layer="91"/>
 <pinref part="P-4" gate="1" pin="V-"/>
 <junction x="134.62" y="91.44"/>
-<pinref part="D8" gate="G$1" pin="A"/>
-<wire x1="119.38" y1="101.6" x2="119.38" y2="91.44" width="0.1524" layer="91"/>
-<junction x="119.38" y="91.44"/>
 </segment>
 <segment>
@@
 <pinref part="OK1" gate="A" pin="EMIT"/>
 <junction x="114.3" y="106.68"/>
-<pinref part="D8" gate="G$1" pin="C"/>
-<junction x="119.38" y="106.68"/>
-</segment>
-</net>
+</segment>
+</net>
