File: eagle/pa97.brd (EAGLE design)
At the start: 152.4 x 152.4 mm, 20 parts

Commit message: pa97 test board
Parts:
- added C6: 10n, rcl:C075-032X103
- added R1, R10, R11, R12, R2, R8, R9: 1M, rcl:0207/10
- added R15: 50k, rcl:0207/10
- added R5, R6, R7: 25k, rcl:0207/10
- added U$5, U$6: 5569-2, con-molex:5569-2
- R3: value 10k -> 25k
- R4: value 300k -> 1M
- moved D9 131.9 mm to (104.4, 71.6)
- moved D1 130.2 mm to (109.7, 48.8)
- moved D10 127.5 mm to (84.1, 77.7)
- moved D2 126.6 mm to (94.5, 53.8), turned to 180 degrees
- moved D8 94.0 mm to (61.5, 67.1), turned to 90 degrees
- moved U$3 87.6 mm to (114.6, 41.1)
- moved D7 84.7 mm to (54.4, 67.1), turned to 270 degrees
- moved C4 42.2 mm to (45.0, 82.0), turned to 270 degrees
- moved C3 41.2 mm to (54.9, 86.4)
- moved U$2 31.0 mm to (15.5, 85.9)
- moved R14 18.4 mm to (25.7, 18.3), turned to 270 degrees
- moved C5 17.8 mm to (77.7, 69.3)
- moved R4 12.9 mm to (73.9, 52.6), turned to 0 degrees
- moved C2 9.23 mm to (20.3, 63.2), turned to 0 degrees
- moved R3 7.50 mm to (56.4, 47.0), turned to 0 degrees
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Connections:
- new net N$10: D7.A, D8.C, R3.2, R4.1, U$4.P$1
- new net N$12: R8.1, R9.2
- new net N$14: R10.2, R9.1
- new net N$15: R10.1, R11.2
- new net N$16: R11.1, R12.2
- new net N$17: R12.1, R15.1, U$5.P$1
- new net N$2: R1.1, R4.2
- new net N$3: R3.1, R5.2
- new net N$4: R5.1, R6.2
- new net N$5: R6.1, R7.1
- net +5V: now also C6.1, U$6.P$1
- net GND: now also C6.2, R15.2, R7.2, U$5.P$2, U$6.P$2; no longer R3.2
- net N$11: now also R2.2, R8.2; no longer R4.2
- net N$8: now also R1.2, R2.1; no longer D7.A, D8.C, R3.1, R4.1, U$4.P$1
Routing:
- net N$13: track 0.00 -> 101.4 mm
- net V+: track 0.00 -> 97.1 mm
- net V-: track 0.00 -> 89.8 mm
- net N$11: track 0.00 -> 85.2 mm
- net -15V: track 0.00 -> 51.0 mm
- net +5V: track 0.00 -> 49.3 mm
- net N$10: track 0.00 -> 33.6 mm
- net +15V: track 0.00 -> 17.8 mm
- net N$17: track 0.00 -> 17.5 mm
- net N$24: track 0.00 -> 15.7 mm
- net N$9: track 0.36 -> 15.8 mm
- net N$16: track 0.00 -> 9.91 mm
- net N$14: track 0.00 -> 9.61 mm
- net N$15: track 0.00 -> 9.25 mm
- net N$12: track 0.00 -> 8.89 mm
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
Commit message: Test layouts pa97
Parts:
- removed D7, D8: 1N4148DO35-10, diode:DO35-10
- removed R3: 25k, rcl:0207/10
- added C7: 10p, rcl:C075-032X103
- added D3, D4: 1n4742, diode:DO41Z10
- added R16, R17: 0, rcl:0207/10
- C5: value 10n -> 10p
- R15: value 50k -> 5k
- R5, R6, R7: value 25k -> 25.5k
- moved U$3 27.3 mm to (141.7, 38.9)
- moved D2 22.5 mm to (113.5, 41.9), turned to 270 degrees
- moved C5 20.3 mm to (77.7, 89.7)
- moved U$2 18.4 mm to (9.91, 103.4)
- moved U$6 18.4 mm to (9.91, 91.7)
- moved C3 17.5 mm to (54.6, 103.9)
- moved C4 17.5 mm to (44.7, 99.6)
- moved D1 17.4 mm to (125.0, 57.1), turned to 90 degrees
- moved D9 17.3 mm to (104.4, 88.9)
- moved D10 17.3 mm to (84.1, 95.0)
- moved R9 10.7 mm to (88.1, 16.0)
- moved R10 10.7 mm to (97.0, 16.0)
- moved R11 10.7 mm to (105.7, 16.0)
- moved U$5 10.7 mm to (133.1, 10.9)
- moved R12 10.7 mm to (115.6, 16.0)
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Connections:
- new net N$18: R16.2, X1.3
- new net N$19: R17.2, X1.2
- new net N$20: D3.C, D4.C
- net GND: now also R16.1, R17.1; no longer X1.2, X1.3
- net N$10: now also C7.1; no longer D7.A, D8.C, R3.2, R4.1, U$4.P$1
- net N$11: now also C7.2
- net N$13: now also D3.A; no longer D7.C, D8.A
- net N$3: now also D4.A, R4.1, U$4.P$1; no longer R3.1
Routing:
- net N$13: track 101.4 -> 147.7 mm
- net N$3: track 6.96 -> 49.4 mm
- net N$11: track 85.2 -> 114.0 mm
- net V+: track 97.1 -> 120.4 mm
- net V-: track 89.8 -> 112.8 mm
- net N$7: track 7.37 -> 27.7 mm
- net N$6: track 8.42 -> 28.7 mm
- net +5V: track 49.3 -> 61.9 mm
- net N$19: track 0.00 -> 8.23 mm
- net N$18: track 0.00 -> 7.64 mm
- net N$20: track 0.00 -> 6.60 mm
- net N$1: track 5.08 -> 11.4 mm
- net N$10: track 33.6 -> 27.7 mm
- net -15V: track 51.0 -> 56.7 mm
- net N$9: track 15.8 -> 18.0 mm
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