File: eagle/pa97.sch (EAGLE design)
At the start: 39 parts, among them IC1 LT1352PA, Q3 C2M0280120D90H, Q4 C2M0280120D90H, T1 2N3904

Commit message: pa 97 circuit
Parts:
- removed D3, D4, D5, D6: P6KEXX, diode:P6KEXX
- removed DC1: (no value), dc-dc-converter:NCS
- removed IC1: LT1352PA, linear-technology:LT1352PA
- removed OK1: PC817, optocoupler:PC817
- removed Q1, Q2: (no value), transistor-power:PMOSFET_NTO220BV
- removed Q3, Q4: C2M0280120D90H, transistor-power:C2M0280120D90H
- removed R1: 65, rcl:R-US_0207/10
- removed R10, R11, R6, R9: 10k, rcl:R-US_0207/10
- removed R12: 20k, rcl:R-US_0207/15
- removed R15, R5, R7: 1M, resistor:R-US_0414/15
- removed R2: 5k, rcl:R-US_0207/10
- removed R8: 50k, rcl:R-US_0207/10
- removed T1: 2N3904, transistor:2N3904
- added D10, D9: P6KEXXA, diode:P6KEXXA
- added D8: 1N4148DO35-10, diode:1N4148DO35-10
- added U$4: PA97, apex:PA97
- D1, D2: value P6KEXX -> P6KEXXA; device diode:P6KEXX -> diode:P6KEXXA
- R3: value 100 -> 10k
- R4: value 100 -> 300k
Connections:
- removed net N$10: D1.A, D7.A, R1.1, R15.2, T1.E, U$3G$1.S
- removed net N$12: IC1A.+IN, R10.1
- removed net N$14: Q2.S, R2.2
- removed net N$16: DC1.VOUT, R6.2
- removed net N$17: C5.1, R9.1
- removed net N$18: IC1A.-IN, R11.1, R9.2
- removed net N$19: C5.2, IC1A.OUT, R12.2
- removed net N$2: D2.C, D3.A
- removed net N$21: R11.2, R7.1, R8.2
- removed net N$22: OK1.COL, R4.2, R6.1
- removed net N$23: R15.1, R7.2
- removed net N$25: OK1.A, R12.1
- removed net N$3: D3.C, D4.C
- removed net N$4: D4.A, D5.C
- removed net N$5: D5.A, D6.C
- net +15V: no longer DC1.VIN+, IC1A.V+
- net -15V: no longer IC1A.V-, OK1.C
- net GND: now also D1.A, D10.C, D9.A, R3.2; no longer D6.A, DC1.VIN-, R8.1
- net N$1: now also D2.C; no longer D2.A
- net N$11: now also D2.A, R4.2, U$3G$1.S, U$4.OUT; no longer Q2.G, R4.1
- net N$13: now also D7.C, D8.A, U$4.+IN; no longer R10.2
- net N$6: now also C5.1, U$4.CC1; no longer Q1.G, R3.1
- net N$7: now also C5.2, U$4.CC2; no longer D7.C, Q2.D, R3.2, R5.1, T1.C
- net N$8: now also D7.A, D8.C, R3.1, R4.1, U$4.-IN; no longer Q1.S, R1.2, T1.B
- net V+: now also D9.C, U$4.V+; no longer Q1.D, R5.2
- net V-: now also D10.A, U$4.V-; no longer DC1.0V, OK1.EMIT, R2.1
Other:
- moved on the sheet: C5, D1, D2, D7, R3, R4, U$1G$4, U$3G$1, U$3G$2

Commit message: pa97 test board
Parts:
- added C6: 10n, rcl:C-US075-032X103
- added R1, R10, R11, R12, R2, R8, R9: 1M, rcl:R-US_0207/10
- added R15: 50k, rcl:R-US_0207/10
- added R5, R6, R7: 25k, rcl:R-US_0207/10
- added U$5, U$6: 5569-2, con-molex:5569-2
- R3: value 10k -> 25k
- R4: value 300k -> 1M
Connections:
- new net N$10: D7.A, D8.C, R3.2, R4.1, U$4.-IN
- new net N$12: R8.1, R9.2
- new net N$14: R10.2, R9.1
- new net N$15: R10.1, R11.2
- new net N$16: R11.1, R12.2
- new net N$17: R12.1, R15.1, U$5G$1.S
- new net N$2: R1.1, R4.2
- new net N$3: R3.1, R5.2
- new net N$4: R5.1, R6.2
- new net N$5: R6.1, R7.1
- net +5V: now also C6.1, U$6G$1.S
- net GND: now also C6.2, R15.2, R7.2, U$5G$2.S, U$6G$2.S; no longer R3.2
- net N$11: now also R2.2, R8.2; no longer R4.2
- net N$8: now also R1.2, R2.1; no longer D7.A, D8.C, R3.1, R4.1, U$4.-IN
Other:
- moved on the sheet: C5, D1, D2, R3, R4, U$3G$1, U$3G$2

Commit message: Test layouts pa97
Parts:
- removed D7, D8: 1N4148DO35-10, diode:1N4148DO35-10
- removed R3: 25k, rcl:R-US_0207/10
- added C7: 10p, rcl:C-US075-032X103
- added D3, D4: 1n4742, diode:ZENER-DIODEDO41Z10
- added R16, R17: 0, rcl:R-US_0207/10
- C5: value 10n -> 10p
- R15: value 50k -> 5k
- R5, R6, R7: value 25k -> 25.5k
Connections:
- new net N$18: R16.2, X1-3.S
- new net N$19: R17.2, X1-2.S
- new net N$20: D3.C, D4.C
- net GND: now also R16.1, R17.1; no longer X1-2.S, X1-3.S
- net N$10: now also C7.1; no longer D7.A, D8.C, R3.2, R4.1, U$4.-IN
- net N$11: now also C7.2
- net N$13: now also D3.A; no longer D7.C, D8.A
- net N$3: now also D4.A, R4.1, U$4.-IN; no longer R3.1
Other:
- moved on the sheet: R13, R14, U$1G$1, U$1G$2, U$1G$4, U$2G$1, U$2G$2, U$2G$3, U$2G$4, U$6G$1, U$6G$2, X1-1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
