File: eagle/regulator_plus_switch_multi.sch (EAGLE design)
At the start: 69 parts, among them IC2 LT1352PA, IC3 DG419DJN, IC4 LT1352PA, J23 5569-2, J26 5569-2, Q1 2N3906, Q2 2N3906, T1 2N3904, T2 2N3904

Commit message: 8chan
Parts:
- added C10, C11, C12, C13, C14, C15, C16, C17, C18, C19, C20, C21, C22, C23: 10p, rcl:C-US075-032X103
- added D1, D11, D12, D15, D16, D19, D20, D23, D24, D27, D28, D31, D32, D4: P6KEXXA, diode:P6KEXXA
- added D13, D14, D17, D18, D21, D22, D25, D26, D29, D30, D33, D34, D5, D6: 1n4742, diode:ZENER-DIODEDO41Z10
- added IC1, IC11, IC13, IC15, IC5, IC7, IC9: LT1352PA, linear-technology:LT1352PA
- added IC10, IC12, IC14, IC16, IC6, IC8: DG419DJN, linear:DG419DJN
- added KK2, KK3, KK4, KK5, KK6, KK7, KK8: SK125/50C247, heatsink:SK125/50C247
- added POT2, POT3, POT4, POT5, POT6, POT7, POT8: 5569-4, con-molex:5569-4
- added R1, R110, R111, R124, R135, R136, R149, R160, R161, R174, R185, R186, R199, R36, R49, R60, R61, R74, R85, R86, R99: 20k, rcl:R-US_0207/15
- added R100, R125, R150, R175, R200, R50, R75: 16k, rcl:R-US_0207/10
- added R101, R126, R151, R176, R201, R51, R76: 12.75k, rcl:R-US_0207/10
- added R102, R112, R114, R123, R127, R137, R139, R148, R152, R162, R164, R173, R177, R187, R189, R198, R202, R37, R39, R48, R52, R62, R64, R73, R77, R87, R89, R98: 10k, rcl:R-US_0207/10
- added R104, R105, R106, R129, R130, R131, R154, R155, R156, R179, R180, R181, R204, R205, R206, R54, R55, R56, R79, R80, R81: 1M, rcl:R-US_0207/10
- added R107, R108, R109, R132, R133, R134, R157, R158, R159, R182, R183, R184, R207, R208, R209, R57, R58, R59, R82, R83, R84: 25.5k, rcl:R-US_0207/10
- added R113, R138, R163, R188, R38, R63, R88: 40k, rcl:R-US_0207/10
- added R115, R140, R165, R190, R40, R65, R90: 17k, rcl:R-US_0207/10
- added R116, R141, R166, R191, R41, R66, R91: 13k, rcl:R-US_0207/10
- added R117, R118, R119, R120, R121, R142, R143, R144, R145, R146, R167, R168, R169, R170, R171, R192, R193, R194, R195, R196, R42, R43, R44, R45, R46, R67, R68, R69, R70, R71, R92, R93, R94, R95, R96: 1M, resistor:R-US_0207/10
- added R122, R147, R172, R197, R47, R72, R97: 100k, rcl:R-US_0207/10
- added U$1, U$2, U$3, U$5, U$6, U$7, U$8: PA97, apex:PA97
- IC4: value LT1352PA -> DG419DJN; device linear-technology:LT1352PA -> linear:DG419DJN
- R26: value 50k -> 100k
- R29: value 17k -> 16k
- R30: value 13k -> 12.75k
- R33: value 9.09k -> 90.9k
- R34: value 1k -> 10k
Connections:
- new net CMD2: EXTERNAL-3.F, R37.2
- new net CMD3: EXTERNAL-5.F, R62.2
- new net CMD4: EXTERNAL-7.F, R87.2
- new net CMD5: EXTERNAL-9.F, R112.2
- new net CMD6: EXTERNAL-11.F, R137.2
- new net CMD7: EXTERNAL-13.F, R162.2
- new net CMD8: EXTERNAL-15.F, R187.2
- new net N$100: POT4G$1.S, R86.2
- new net N$101: C14.1, U$3.CC1
- new net N$102: C14.2, U$3.CC2
- new net N$103: C15.2, D16.A, OUTG$4.P$1, R106.2, R92.2, U$3.OUT
- new net N$104: D15.C, D16.C
- new net N$105: R104.2, R105.1
- new net N$106: R107.1, R108.2
- new net N$107: R108.1, R109.1
- new net N$108: R105.2, R106.1
- new net N$109: D17.C, D18.C
- new net N$110: IC9A.-IN, R112.1, R113.2
- new net N$111: IC9A.+IN, R114.1
- new net N$112: R114.2, R115.2, R116.1
- new net N$113: IC10A.S2, IC9A.OUT, R113.1
- new net N$114: R117.1, R118.2
- new net N$115: R118.1, R119.2
- new net N$116: R119.1, R120.2
- new net N$117: R120.1, R121.2
- new net N$118: DISPLAYG$5.S, R121.1, R122.2, R124.2
- new net N$119: EXTERNAL-21.F, IC9B.OUT, R123.1
- new net N$120: R125.2, R126.1, R127.2
- new net N$121: IC9B.-IN, R127.1
- new net N$122: IC9B.+IN, R123.2, R124.1
- new net N$123: POT5G$2.S, R110.2
- new net N$124: IC10A.S1, POT5G$4.S
- new net N$125: POT5G$1.S, R111.2
- new net N$126: C16.1, U$5.CC1
- new net N$127: C16.2, U$5.CC2
- new net N$128: C17.2, D20.A, OUTG$5.P$1, R117.2, R131.2, U$5.OUT
- new net N$129: D19.C, D20.C
- new net N$130: R129.2, R130.1
- new net N$131: R132.1, R133.2
- new net N$132: R133.1, R134.1
- new net N$133: R130.2, R131.1
- new net N$134: D21.C, D22.C
- new net N$135: IC11A.-IN, R137.1, R138.2
- new net N$136: IC11A.+IN, R139.1
- new net N$137: R139.2, R140.2, R141.1
- new net N$138: IC11A.OUT, IC12A.S2, R138.1
- new net N$139: R142.1, R143.2
- new net N$140: R143.1, R144.2
- new net N$141: R144.1, R145.2
- new net N$142: R145.1, R146.2
- new net N$143: DISPLAYG$6.S, R146.1, R147.2, R149.2
- new net N$144: EXTERNAL-22.F, IC11B.OUT, R148.1
- new net N$145: R150.2, R151.1, R152.2
- new net N$146: IC11B.-IN, R152.1
- new net N$147: IC11B.+IN, R148.2, R149.1
- new net N$148: POT6G$2.S, R135.2
- new net N$149: IC12A.S1, POT6G$4.S
- new net N$150: POT6G$1.S, R136.2
- new net N$151: C18.1, U$6.CC1
- new net N$152: C18.2, U$6.CC2
- new net N$153: C19.2, D24.A, OUTG$6.P$1, R142.2, R156.2, U$6.OUT
- new net N$154: D23.C, D24.C
- new net N$155: R154.2, R155.1
- new net N$156: R157.1, R158.2
- new net N$157: R158.1, R159.1
- new net N$158: R155.2, R156.1
- new net N$159: D25.C, D26.C
- new net N$160: IC13A.-IN, R162.1, R163.2
- new net N$161: IC13A.+IN, R164.1
- new net N$162: R164.2, R165.2, R166.1
- new net N$163: IC13A.OUT, IC14A.S2, R163.1
- new net N$164: R167.1, R168.2
- new net N$165: R168.1, R169.2
- new net N$166: R169.1, R170.2
- new net N$167: R170.1, R171.2
- new net N$168: DISPLAYG$7.S, R171.1, R172.2, R174.2
- new net N$169: EXTERNAL-23.F, IC13B.OUT, R173.1
- new net N$170: R175.2, R176.1, R177.2
- new net N$171: IC13B.-IN, R177.1
- new net N$172: IC13B.+IN, R173.2, R174.1
- new net N$173: POT7G$2.S, R160.2
- new net N$174: IC14A.S1, POT7G$4.S
- new net N$175: POT7G$1.S, R161.2
- new net N$176: C20.1, U$7.CC1
- new net N$177: C20.2, U$7.CC2
- new net N$178: C21.2, D28.A, OUTG$7.P$1, R167.2, R181.2, U$7.OUT
- new net N$179: D27.C, D28.C
- new net N$180: R179.2, R180.1
- new net N$181: R182.1, R183.2
- new net N$182: R183.1, R184.1
- new net N$183: R180.2, R181.1
- new net N$184: D29.C, D30.C
- new net N$185: IC15A.-IN, R187.1, R188.2
- new net N$186: IC15A.+IN, R189.1
- new net N$187: R189.2, R190.2, R191.1
- new net N$188: IC15A.OUT, IC16A.S2, R188.1
- new net N$189: R192.1, R193.2
- new net N$190: R193.1, R194.2
- new net N$191: R194.1, R195.2
- new net N$192: R195.1, R196.2
- new net N$193: DISPLAYG$8.S, R196.1, R197.2, R199.2
- new net N$194: EXTERNAL-24.F, IC15B.OUT, R198.1
- new net N$195: R200.2, R201.1, R202.2
- new net N$196: IC15B.-IN, R202.1
- new net N$197: IC15B.+IN, R198.2, R199.1
- new net N$198: POT8G$2.S, R185.2
- new net N$199: IC16A.S1, POT8G$4.S
- new net N$200: POT8G$1.S, R186.2
- new net N$201: C22.1, U$8.CC1
- new net N$202: C22.2, U$8.CC2
- new net N$203: C23.2, D32.A, OUTG$8.P$1, R192.2, R206.2, U$8.OUT
- new net N$204: D31.C, D32.C
- new net N$205: R204.2, R205.1
- new net N$206: R207.1, R208.2
- new net N$207: R208.1, R209.1
- new net N$208: R205.2, R206.1
- new net N$209: D33.C, D34.C
- new net N$23: R39.2, R40.2, R41.1
- new net N$28: IC1A.OUT, IC4A.S2, R38.1
- new net N$38: R42.1, R43.2
- new net N$40: R43.1, R44.2
- new net N$41: R44.1, R45.2
- new net N$42: R45.1, R46.2
- new net N$43: DISPLAYG$2.S, R46.1, R47.2, R49.2
- new net N$44: EXTERNAL-18.F, IC1B.OUT, R48.1
- new net N$45: R50.2, R51.1, R52.2
- new net N$46: IC1B.-IN, R52.1
- new net N$47: IC1B.+IN, R48.2, R49.1
- new net N$48: POT2G$2.S, R1.2
- new net N$49: IC4A.S1, POT2G$4.S
- new net N$50: POT2G$1.S, R36.2
- new net N$51: C10.1, U$1.CC1
- new net N$52: C10.2, U$1.CC2
- new net N$53: C11.2, D4.A, OUTG$2.P$1, R42.2, R56.2, U$1.OUT
- new net N$54: D1.C, D4.C
- new net N$55: R54.2, R55.1
- new net N$56: R57.1, R58.2
- new net N$57: R58.1, R59.1
- new net N$58: R55.2, R56.1
- new net N$59: D5.C, D6.C
- new net N$6: IC1A.-IN, R37.1, R38.2
- new net N$60: IC5A.-IN, R62.1, R63.2
- new net N$61: IC5A.+IN, R64.1
- new net N$62: R64.2, R65.2, R66.1
- new net N$63: IC5A.OUT, IC6A.S2, R63.1
- new net N$64: R67.1, R68.2
- new net N$65: R68.1, R69.2
- new net N$66: R69.1, R70.2
- new net N$67: R70.1, R71.2
- new net N$68: DISPLAYG$3.S, R71.1, R72.2, R74.2
- new net N$69: EXTERNAL-19.F, IC5B.OUT, R73.1
- new net N$7: IC1A.+IN, R39.1
- new net N$70: R75.2, R76.1, R77.2
- new net N$71: IC5B.-IN, R77.1
- new net N$72: IC5B.+IN, R73.2, R74.1
- new net N$73: POT3G$2.S, R60.2
- new net N$74: IC6A.S1, POT3G$4.S
- new net N$75: POT3G$1.S, R61.2
- new net N$76: C12.1, U$2.CC1
- new net N$77: C12.2, U$2.CC2
- new net N$78: C13.2, D12.A, OUTG$3.P$1, R67.2, R81.2, U$2.OUT
- new net N$79: D11.C, D12.C
- new net N$80: R79.2, R80.1
- new net N$81: R82.1, R83.2
- new net N$82: R83.1, R84.1
- new net N$83: R80.2, R81.1
- new net N$84: D13.C, D14.C
- new net N$85: IC7A.-IN, R87.1, R88.2
- new net N$86: IC7A.+IN, R89.1
- new net N$87: R89.2, R90.2, R91.1
- new net N$88: IC7A.OUT, IC8A.S2, R88.1
- new net N$89: R92.1, R93.2
- new net N$90: R93.1, R94.2
- new net N$91: R94.1, R95.2
- new net N$92: R95.1, R96.2
- new net N$93: DISPLAYG$4.S, R96.1, R97.2, R99.2
- new net N$94: EXTERNAL-20.F, IC7B.OUT, R98.1
- new net N$95: R100.2, R101.1, R102.2
- new net N$96: IC7B.-IN, R102.1
- new net N$97: IC7B.+IN, R98.2, R99.1
- new net N$98: POT4G$2.S, R85.2
- new net N$99: IC8A.S1, POT4G$4.S
- net +15V: now also IC10P.V+, IC11A.V+, IC12P.V+, IC13A.V+, IC14P.V+, IC15A.V+, IC16P.V+, IC1A.V+, IC4P.V+, IC5A.V+, IC6P.V+, IC7A.V+, IC8P.V+, IC9A.V+, R1.1, R101.2, R110.1, R116.2, R126.2, R135.1, R141.2, R151.2, R160.1, R166.2, R176.2, R185.1, R191.2, R201.2, R41.2, R51.2, R60.1, R66.2, R76.2, R85.1, R91.2; no longer IC4A.V+
- net +5V: now also IC10VL.VL, IC12VL.VL, IC14VL.VL, IC16VL.VL, IC4VL.VL, IC6VL.VL, IC8VL.VL
- net -15V: now also IC10P.V-, IC11A.V-, IC12P.V-, IC13A.V-, IC14P.V-, IC15A.V-, IC16P.V-, IC1A.V-, IC4P.V-, IC5A.V-, IC6P.V-, IC7A.V-, IC8P.V-, IC9A.V-, R100.1, R111.1, R115.1, R125.1, R136.1, R140.1, R150.1, R161.1, R165.1, R175.1, R186.1, R190.1, R200.1, R36.1, R40.1, R50.1, R61.1, R65.1, R75.1, R86.1, R90.1; no longer IC4A.V-
- net GND: now also D1.A, D11.A, D15.A, D19.A, D23.A, D27.A, D31.A, IC10P.GND, IC12P.GND, IC14P.GND, IC16P.GND, IC4P.GND, IC6P.GND, IC8P.GND, R109.2, R122.1, R134.2, R147.1, R159.2, R172.1, R184.2, R197.1, R209.2, R47.1, R59.2, R72.1, R84.2, R97.1
- net MAN: now also IC10A.IN, IC12A.IN, IC14A.IN, IC16A.IN, IC4A.IN, IC6A.IN, IC8A.IN
- net N$35: now also IC2B.OUT; no longer IC4A.OUT
- net N$37: now also IC2B.-IN; no longer IC4A.+IN
- net N$39: now also IC2B.+IN; no longer IC4A.-IN
- net V+_SAFE: now also U$1.V+, U$2.V+, U$3.V+, U$5.V+, U$6.V+, U$7.V+, U$8.V+
- net V-_SAFE: now also U$1.V-, U$2.V-, U$3.V-, U$5.V-, U$6.V-, U$7.V-, U$8.V-
- net VIN+: now also D13.A, D17.A, D21.A, D25.A, D29.A, D33.A, D5.A, IC10A.D, IC12A.D, IC14A.D, IC16A.D, IC4A.D, IC6A.D, IC8A.D, U$1.+IN, U$2.+IN, U$3.+IN, U$5.+IN, U$6.+IN, U$7.+IN, U$8.+IN
- net VIN-: now also C11.1, C13.1, C15.1, C17.1, C19.1, C21.1, C23.1, D14.A, D18.A, D22.A, D26.A, D30.A, D34.A, D6.A, R104.1, R107.2, R129.1, R132.2, R154.1, R157.2, R179.1, R182.2, R204.1, R207.2, R54.1, R57.2, R79.1, R82.2, U$1.-IN, U$2.-IN, U$3.-IN, U$5.-IN, U$6.-IN, U$7.-IN, U$8.-IN
Other:
- moved on the sheet: C1, C2, C3, C4, C5, C6, C7, C8, C9, D10, D2, D3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

Commit message: 8chan
Parts:
- R1, R110, R111, R124, R13, R135, R136, R14, R149, R160, R161, R174, R185, R186, R199, R28, R32, R36, R49, R60, R61, R74, R85, R86, R99: device rcl:R-US_0207/15 -> rcl:R-US_0207/10

Commit message: submit 8 chan
Parts:
- C8, C9: value cc -> 1n
- Q1, Q2: value 2N3906 -> STX616-AP
- R10, R12: value rb -> 1k
- R11, R8: value rlim -> 68
- R15, R9: value rl -> 4.99M
- T1, T2: value 2N3904 -> ZTX560
Changed lines of the file:
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@@
 <grid distance="0.1" unitdist="inch" unit="inch" style="lines" multiple="1" display="no" altdistance="0.01" altunitdist="inch" altunit="inch"/>
 <layers>
-<layer number="1" name="Top" color="4" fill="1" visible="yes" active="no"/>
-<layer number="2" name="Route2" color="1" fill="3" visible="yes" active="no"/>
-<layer number="3" name="Route3" color="4" fill="3" visible="yes" active="no"/>
-<layer number="4" name="Route4" color="1" fill="4" visible="yes" active="no"/>
-<layer number="5" name="Route5" color="4" fill="4" visible="yes" active="no"/>
-<layer number="6" name="Route6" color="1" fill="8" visible="yes" active="no"/>
-<layer number="7" name="Route7" color="4" fill="8" visible="yes" active="no"/>
-<layer number="8" name="Route8" color="1" fill="2" visible="yes" active="no"/>
-<layer number="9" name="Route9" color="4" fill="2" visible="yes" active="no"/>
-<layer number="10" name="Route10" color="1" fill="7" visible="yes" active="no"/>
-<layer number="11" name="Route11" color="4" fill="7" visible="yes" active="no"/>
-<layer number="12" name="Route12" color="1" fill="5" visible="yes" active="no"/>
-<layer number="13" name="Route13" color="4" fill="5" visible="yes" active="no"/>
-<layer number="14" name="Route14" color="1" fill="6" visible="yes" active="no"/>
-<layer number="15" name="Route15" color="4" fill="6" visible="yes" active="no"/>
-<layer number="16" name="Bottom" color="1" fill="1" visible="yes" active="no"/>
-<layer number="17" name="Pads" color="2" fill="1" visible="yes" active="no"/>
-<layer number="18" name="Vias" color="2" fill="1" visible="yes" active="no"/>
-<layer number="19" name="Unrouted" color="6" fill="1" visible="yes" active="no"/>
-<layer number="20" name="Dimension" color="15" fill="1" visible="yes" active="no"/>
-<layer number="21" name="tPlace" color="7" fill="1" visible="yes" active="no"/>
-<layer number="22" name="bPlace" color="7" fill="1" visible="yes" active="no"/>
-<layer number="23" name="tOrigins" color="15" fill="1" visible="yes" active="no"/>
-<layer number="24" name="bOrigins" color="15" fill="1" visible="yes" active="no"/>
-<layer number="25" name="tNames" color="7" fill="1" visible="yes" active="no"/>
-<layer number="26" name="bNames" color="7" fill="1" visible="yes" active="no"/>
-<layer number="27" name="tValues" color="7" fill="1" visible="yes" active="no"/>
-<layer number="28" name="bValues" color="7" fill="1" visible="yes" active="no"/>
+<layer number="1" name="Top" color="4" fill="1" visible="no" active="no"/>
+<layer number="2" name="Route2" color="1" fill="3" visible="no" active="no"/>
+<layer number="3" name="Route3" color="4" fill="3" visible="no" active="no"/>
+<layer number="4" name="Route4" color="1" fill="4" visible="no" active="no"/>
+<layer number="5" name="Route5" color="4" fill="4" visible="no" active="no"/>
+<layer number="6" name="Route6" color="1" fill="8" visible="no" active="no"/>
+<layer number="7" name="Route7" color="4" fill="8" visible="no" active="no"/>
+<layer number="8" name="Route8" color="1" fill="2" visible="no" active="no"/>
+<layer number="9" name="Route9" color="4" fill="2" visible="no" active="no"/>
+<layer number="10" name="Route10" color="1" fill="7" visible="no" active="no"/>
+<layer number="11" name="Route11" color="4" fill="7" visible="no" active="no"/>
+<layer number="12" name="Route12" color="1" fill="5" visible="no" active="no"/>
+<layer number="13" name="Route13" color="4" fill="5" visible="no" active="no"/>
+<layer number="14" name="Route14" color="1" fill="6" visible="no" active="no"/>
+<layer number="15" name="Route15" color="4" fill="6" visible="no" active="no"/>
+<layer number="16" name="Bottom" color="1" fill="1" visible="no" active="no"/>
+<layer number="17" name="Pads" color="2" fill="1" visible="no" active="no"/>
+<layer number="18" name="Vias" color="2" fill="1" visible="no" active="no"/>
+<layer number="19" name="Unrouted" color="6" fill="1" visible="no" active="no"/>
+<layer number="20" name="Dimension" color="15" fill="1" visible="no" active="no"/>
+<layer number="21" name="tPlace" color="7" fill="1" visible="no" active="no"/>
+<layer number="22" name="bPlace" color="7" fill="1" visible="no" active="no"/>
+<layer number="23" name="tOrigins" color="15" fill="1" visible="no" active="no"/>
+<layer number="24" name="bOrigins" color="15" fill="1" visible="no" active="no"/>
+<layer number="25" name="tNames" color="7" fill="1" visible="no" active="no"/>
+<layer number="26" name="bNames" color="7" fill="1" visible="no" active="no"/>
+<layer number="27" name="tValues" color="7" fill="1" visible="no" active="no"/>
+<layer number="28" name="bValues" color="7" fill="1" visible="no" active="no"/>
 <layer number="29" name="tStop" color="7" fill="3" visible="no" active="no"/>
 <layer number="30" name="bStop" color="7" fill="6" visible="no" active="no"/>
@@
 <layer number="35" name="tGlue" color="7" fill="4" visible="no" active="no"/>
 <layer number="36" name="bGlue" color="7" fill="5" visible="no" active="no"/>
-<layer number="37" name="tTest" color="7" fill="1" visible="yes" active="no"/>
-<layer number="38" name="bTest" color="7" fill="1" visible="yes" active="no"/>
+<layer number="37" name="tTest" color="7" fill="1" visible="no" active="no"/>
+<layer number="38" name="bTest" color="7" fill="1" visible="no" active="no"/>
 <layer number="39" name="tKeepout" color="4" fill="11" visible="no" active="no"/>
 <layer number="40" name="bKeepout" color="1" fill="11" visible="no" active="no"/>
@@
 <layer number="44" name="Drills" color="7" fill="1" visible="no" active="no"/>
 <layer number="45" name="Holes" color="7" fill="1" visible="no" active="no"/>
-<layer number="46" name="Milling" color="3" fill="1" visible="yes" active="no"/>
-<layer number="47" name="Measures" color="7" fill="1" visible="yes" active="no"/>
-<layer number="48" name="Document" color="7" fill="1" visible="yes" active="no"/>
-<layer number="49" name="Reference" color="7" fill="1" visible="yes" active="no"/>
-<layer number="51" name="tDocu" color="7" fill="1" visible="yes" active="no"/>
-<layer number="52" name="bDocu" color="7" fill="1" visible="yes" active="no"/>
+<layer number="46" name="Milling" color="3" fill="1" visible="no" active="no"/>
+<layer number="47" name="Measures" color="7" fill="1" visible="no" active="no"/>
+<layer number="48" name="Document" color="7" fill="1" visible="no" active="no"/>
+<layer number="49" name="Reference" color="7" fill="1" visible="no" active="no"/>
+<layer number="51" name="tDocu" color="7" fill="1" visible="no" active="no"/>
+<layer number="52" name="bDocu" color="7" fill="1" visible="no" active="no"/>
 <layer number="90" name="Modules" color="5" fill="1" visible="yes" active="yes"/>
 <layer number="91" name="Nets" color="2" fill="1" visible="yes" active="yes"/>
@@
 <clearance class="0" value="0.254"/>
 </class>
-<class number="1" name="ground" width="1.016" drill="0">
+<class number="1" name="ground" width="0.6096" drill="0">
 <clearance class="1" value="0.254"/>
 </class>
@@
 <part name="C6" library="rcl" deviceset="C-US" device="075-032X103" value="10n"/>
 <part name="GND6" library="supply1" deviceset="GND" device=""/>
-<part name="T1" library="transistor" deviceset="2N3904" device=""/>
-<part name="T2" library="transistor" deviceset="2N3904" device=""/>
-<part name="Q1" library="transistor-pnp" deviceset="2N3906" device=""/>
-<part name="Q2" library="transistor-pnp" deviceset="2N3906" device=""/>
-<part name="R8" library="rcl" deviceset="R-US_" device="0207/10" value="rlim"/>
-<part name="R9" library="rcl" deviceset="R-US_" device="0207/10" value="rl"/>
-<part name="R10" library="rcl" deviceset="R-US_" device="0207/10" value="rb"/>
-<part name="C8" library="rcl" deviceset="C-US" device="075-032X103" value="cc"/>
+<part name="T1" library="transistor" deviceset="2N3904" device="" value="ZTX560"/>
+<part name="T2" library="transistor" deviceset="2N3904" device="" value="ZTX560"/>
+<part name="Q1" library="transistor-pnp" deviceset="2N3906" device="" value="STX616-AP"/>
+<part name="Q2" library="transistor-pnp" deviceset="2N3906" device="" value="STX616-AP"/>
+<part name="R8" library="rcl" deviceset="R-US_" device="0207/10" value="68"/>
+<part name="R9" library="rcl" deviceset="R-US_" device="0207/10" value="4.99M"/>
+<part name="R10" library="rcl" deviceset="R-US_" device="0207/10" value="1k"/>
+<part name="C8" library="rcl" deviceset="C-US" device="075-032X103" value="1n"/>
 <part name="GND29" library="supply1" deviceset="GND" device=""/>
 <part name="P+20" library="supply1" deviceset="V+" device=""/>
 <part name="P-4" library="supply1" deviceset="V-" device=""/>
-<part name="R11" library="rcl" deviceset="R-US_" device="0207/10" value="rlim"/>
-<part name="R12" library="rcl" deviceset="R-US_" device="0207/10" value="rb"/>
-<part name="C9" library="rcl" deviceset="C-US" device="075-032X103" value="cc"/>
-<part name="R15" library="rcl" deviceset="R-US_" device="0207/10" value="rl"/>
+<part name="R11" library="rcl" deviceset="R-US_" device="0207/10" value="68"/>
+<part name="R12" library="rcl" deviceset="R-US_" device="0207/10" value="1k"/>
+<part name="C9" library="rcl" deviceset="C-US" device="075-032X103" value="1n"/>
+<part name="R15" library="rcl" deviceset="R-US_" device="0207/10" value="4.99M"/>
 <part name="GND31" library="supply1" deviceset="GND" device=""/>
 <part name="DISPLAY1" library="con-molex" deviceset="5569-2" device=""/>
