File: eagle/regulator_plus_switch_multi.brd (EAGLE design)
At the start: 152.7 x 152.4 mm, 69 parts, among them IC2 LT1352PA, IC3 DG419DJN, IC4 LT1352PA, J23 5569-2, J26 5569-2, Q1 2N3906, Q2 2N3906, T1 2N3904, T2 2N3904

Commit message: big board
Parts:
- moved EXTERNAL 308.5 mm to (86.1, 280.2), turned to 0 degrees
- moved OUT 199.8 mm to (152.7, 276.6), turned to 0 degrees
Routing:
- net N$34: track 234.2 -> 0.00 mm
- net +5V: track 219.8 -> 0.00 mm, vias 4 -> 0
- net V-: track 209.8 -> 0.00 mm
- net -15V: track 207.5 -> 0.00 mm, vias 2 -> 0
- net +15V: track 152.9 -> 0.00 mm, vias 2 -> 0
- net N$13: track 145.5 -> 0.00 mm, vias 2 -> 0
- net VIN-: track 144.2 -> 0.00 mm
- net V+: track 137.5 -> 0.00 mm
- net MAN: track 134.7 -> 0.00 mm, vias 2 -> 0
- net VIN+: track 111.3 -> 0.00 mm, vias 2 -> 0
- net N$11: track 84.9 -> 0.00 mm
- net V-_SAFE: track 75.8 -> 0.00 mm
- net N$39: track 41.2 -> 0.00 mm
- net GND: track 40.6 -> 0.00 mm, vias 2 -> 0
- net V+_SAFE: track 36.4 -> 0.00 mm, vias 2 -> 0
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Other:
- board size 152.7 x 152.4 mm -> 215.9 x 292.1 mm

Commit message: 8chan
Parts:
- added C10, C11, C12, C13, C14, C15, C16, C17, C18, C19, C20, C21, C22, C23: 10p, rcl:C075-032X103
- added D1, D11, D12, D15, D16, D19, D20, D23, D24, D27, D28, D31, D32, D4: P6KEXXA, diode:C1702-15
- added D13, D14, D17, D18, D21, D22, D25, D26, D29, D30, D33, D34, D5, D6: 1n4742, diode:DO41Z10
- added IC1, IC11, IC13, IC15, IC5, IC7, IC9: LT1352PA, linear-technology:DIL08
- added IC10, IC12, IC14, IC16, IC6, IC8: DG419DJN, linear:DIL08
- added KK2, KK3, KK4, KK5, KK6, KK7, KK8: SK125/50C247, heatsink:C247-050
- added POT2, POT3, POT4, POT5, POT6, POT7, POT8: 5569-4, con-molex:5669-4
- added R1, R110, R111, R124, R135, R136, R149, R160, R161, R174, R185, R186, R199, R36, R49, R60, R61, R74, R85, R86, R99: 20k, rcl:0207/15
- added R100, R125, R150, R175, R200, R50, R75: 16k, rcl:0207/10
- added R101, R126, R151, R176, R201, R51, R76: 12.75k, rcl:0207/10
- added R102, R112, R114, R123, R127, R137, R139, R148, R152, R162, R164, R173, R177, R187, R189, R198, R202, R37, R39, R48, R52, R62, R64, R73, R77, R87, R89, R98: 10k, rcl:0207/10
- added R104, R105, R106, R129, R130, R131, R154, R155, R156, R179, R180, R181, R204, R205, R206, R54, R55, R56, R79, R80, R81: 1M, rcl:0207/10
- added R107, R108, R109, R132, R133, R134, R157, R158, R159, R182, R183, R184, R207, R208, R209, R57, R58, R59, R82, R83, R84: 25.5k, rcl:0207/10
- added R113, R138, R163, R188, R38, R63, R88: 40k, rcl:0207/10
- added R115, R140, R165, R190, R40, R65, R90: 17k, rcl:0207/10
- added R116, R141, R166, R191, R41, R66, R91: 13k, rcl:0207/10
- added R117, R118, R119, R120, R121, R142, R143, R144, R145, R146, R167, R168, R169, R170, R171, R192, R193, R194, R195, R196, R42, R43, R44, R45, R46, R67, R68, R69, R70, R71, R92, R93, R94, R95, R96: 1M, resistor:0207/10
- added R122, R147, R172, R197, R47, R72, R97: 100k, rcl:0207/10
- added U$1, U$2, U$3, U$5, U$6, U$7, U$8: PA97, apex:7SIP
- IC4: value LT1352PA -> DG419DJN; device linear-technology:DIL08 -> linear:DIL08
- R26: value 50k -> 100k
- R29: value 17k -> 16k
- R30: value 13k -> 12.75k
- R33: value 9.09k -> 90.9k
- R34: value 1k -> 10k
- moved POWER 209.9 mm to (9.91, 262.4), turned to 270 degrees
- moved HVIN 207.3 mm to (201.9, 4.83), turned to 0 degrees
- moved C1 204.3 mm to (24.9, 272.3), turned to 0 degrees
- moved C6 192.9 mm to (25.1, 260.1), turned to 0 degrees
- moved C2 186.0 mm to (25.7, 252.2), turned to 0 degrees
- moved C3 181.1 mm to (202.7, 32.8), turned to 180 degrees
- moved D2 179.8 mm to (198.9, 25.4), turned to 180 degrees
- moved DISPLAY 166.6 mm to (9.91, 211.8)
- moved R32 160.9 mm to (59.9, 216.2), turned to 180 degrees
- moved C4 132.4 mm to (148.1, 22.4), turned to 180 degrees
- moved Q2 130.1 mm to (180.8, 21.6), turned to 180 degrees
- moved R8 120.3 mm to (177.0, 33.3), turned to 0 degrees
- moved D3 119.5 mm to (144.3, 29.0), turned to 0 degrees
- moved T1 116.9 mm to (126.7, 23.1), turned to 180 degrees
- moved R10 116.7 mm to (172.0, 24.9), turned to 90 degrees
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Connections:
- new net CMD2: EXTERNAL.3, R37.2
- new net CMD3: EXTERNAL.5, R62.2
- new net CMD4: EXTERNAL.7, R87.2
- new net CMD5: EXTERNAL.9, R112.2
- new net CMD6: EXTERNAL.11, R137.2
- new net CMD7: EXTERNAL.13, R162.2
- new net CMD8: EXTERNAL.15, R187.2
- new net N$100: POT4.P$1, R86.2
- new net N$101: C14.1, U$3.P$3
- new net N$102: C14.2, U$3.P$4
- new net N$103: C15.2, D16.A, OUT.P$4, R106.2, R92.2, U$3.P$5
- new net N$104: D15.C, D16.C
- new net N$105: R104.2, R105.1
- new net N$106: R107.1, R108.2
- new net N$107: R108.1, R109.1
- new net N$108: R105.2, R106.1
- new net N$109: D17.C, D18.C
- new net N$110: IC9.2, R112.1, R113.2
- new net N$111: IC9.3, R114.1
- new net N$112: R114.2, R115.2, R116.1
- new net N$113: IC10.8, IC9.1, R113.1
- new net N$114: R117.1, R118.2
- new net N$115: R118.1, R119.2
- new net N$116: R119.1, R120.2
- new net N$117: R120.1, R121.2
- new net N$118: DISPLAY.P$5, R121.1, R122.2, R124.2
- new net N$119: EXTERNAL.21, IC9.7, R123.1
- new net N$120: R125.2, R126.1, R127.2
- new net N$121: IC9.6, R127.1
- new net N$122: IC9.5, R123.2, R124.1
- new net N$123: POT5.P$2, R110.2
- new net N$124: IC10.2, POT5.P$4
- new net N$125: POT5.P$1, R111.2
- new net N$126: C16.1, U$5.P$3
- new net N$127: C16.2, U$5.P$4
- new net N$128: C17.2, D20.A, OUT.P$5, R117.2, R131.2, U$5.P$5
- new net N$129: D19.C, D20.C
- new net N$130: R129.2, R130.1
- new net N$131: R132.1, R133.2
- new net N$132: R133.1, R134.1
- new net N$133: R130.2, R131.1
- new net N$134: D21.C, D22.C
- new net N$135: IC11.2, R137.1, R138.2
- new net N$136: IC11.3, R139.1
- new net N$137: R139.2, R140.2, R141.1
- new net N$138: IC11.1, IC12.8, R138.1
- new net N$139: R142.1, R143.2
- new net N$140: R143.1, R144.2
- new net N$141: R144.1, R145.2
- new net N$142: R145.1, R146.2
- new net N$143: DISPLAY.P$6, R146.1, R147.2, R149.2
- new net N$144: EXTERNAL.22, IC11.7, R148.1
- new net N$145: R150.2, R151.1, R152.2
- new net N$146: IC11.6, R152.1
- new net N$147: IC11.5, R148.2, R149.1
- new net N$148: POT6.P$2, R135.2
- new net N$149: IC12.2, POT6.P$4
- new net N$150: POT6.P$1, R136.2
- new net N$151: C18.1, U$6.P$3
- new net N$152: C18.2, U$6.P$4
- new net N$153: C19.2, D24.A, OUT.P$6, R142.2, R156.2, U$6.P$5
- new net N$154: D23.C, D24.C
- new net N$155: R154.2, R155.1
- new net N$156: R157.1, R158.2
- new net N$157: R158.1, R159.1
- new net N$158: R155.2, R156.1
- new net N$159: D25.C, D26.C
- new net N$160: IC13.2, R162.1, R163.2
- new net N$161: IC13.3, R164.1
- new net N$162: R164.2, R165.2, R166.1
- new net N$163: IC13.1, IC14.8, R163.1
- new net N$164: R167.1, R168.2
- new net N$165: R168.1, R169.2
- new net N$166: R169.1, R170.2
- new net N$167: R170.1, R171.2
- new net N$168: DISPLAY.P$7, R171.1, R172.2, R174.2
- new net N$169: EXTERNAL.23, IC13.7, R173.1
- new net N$170: R175.2, R176.1, R177.2
- new net N$171: IC13.6, R177.1
- new net N$172: IC13.5, R173.2, R174.1
- new net N$173: POT7.P$2, R160.2
- new net N$174: IC14.2, POT7.P$4
- new net N$175: POT7.P$1, R161.2
- new net N$176: C20.1, U$7.P$3
- new net N$177: C20.2, U$7.P$4
- new net N$178: C21.2, D28.A, OUT.P$7, R167.2, R181.2, U$7.P$5
- new net N$179: D27.C, D28.C
- new net N$180: R179.2, R180.1
- new net N$181: R182.1, R183.2
- new net N$182: R183.1, R184.1
- new net N$183: R180.2, R181.1
- new net N$184: D29.C, D30.C
- new net N$185: IC15.2, R187.1, R188.2
- new net N$186: IC15.3, R189.1
- new net N$187: R189.2, R190.2, R191.1
- new net N$188: IC15.1, IC16.8, R188.1
- new net N$189: R192.1, R193.2
- new net N$190: R193.1, R194.2
- new net N$191: R194.1, R195.2
- new net N$192: R195.1, R196.2
- new net N$193: DISPLAY.P$8, R196.1, R197.2, R199.2
- new net N$194: EXTERNAL.24, IC15.7, R198.1
- new net N$195: R200.2, R201.1, R202.2
- new net N$196: IC15.6, R202.1
- new net N$197: IC15.5, R198.2, R199.1
- new net N$198: POT8.P$2, R185.2
- new net N$199: IC16.2, POT8.P$4
- new net N$200: POT8.P$1, R186.2
- new net N$201: C22.1, U$8.P$3
- new net N$202: C22.2, U$8.P$4
- new net N$203: C23.2, D32.A, OUT.P$8, R192.2, R206.2, U$8.P$5
- new net N$204: D31.C, D32.C
- new net N$205: R204.2, R205.1
- new net N$206: R207.1, R208.2
- new net N$207: R208.1, R209.1
- new net N$208: R205.2, R206.1
- new net N$209: D33.C, D34.C
- new net N$23: R39.2, R40.2, R41.1
- new net N$28: IC1.1, IC4.8, R38.1
- new net N$38: R42.1, R43.2
- new net N$40: R43.1, R44.2
- new net N$41: R44.1, R45.2
- new net N$42: R45.1, R46.2
- new net N$43: DISPLAY.P$2, R46.1, R47.2, R49.2
- new net N$44: EXTERNAL.18, IC1.7, R48.1
- new net N$45: R50.2, R51.1, R52.2
- new net N$46: IC1.6, R52.1
- new net N$47: IC1.5, R48.2, R49.1
- new net N$48: POT2.P$2, R1.2
- new net N$49: IC4.2, POT2.P$4
- new net N$50: POT2.P$1, R36.2
- new net N$51: C10.1, U$1.P$3
- new net N$52: C10.2, U$1.P$4
- new net N$53: C11.2, D4.A, OUT.P$2, R42.2, R56.2, U$1.P$5
- new net N$54: D1.C, D4.C
- new net N$55: R54.2, R55.1
- new net N$56: R57.1, R58.2
- new net N$57: R58.1, R59.1
- new net N$58: R55.2, R56.1
- new net N$59: D5.C, D6.C
- new net N$6: IC1.2, R37.1, R38.2
- new net N$60: IC5.2, R62.1, R63.2
- new net N$61: IC5.3, R64.1
- new net N$62: R64.2, R65.2, R66.1
- new net N$63: IC5.1, IC6.8, R63.1
- new net N$64: R67.1, R68.2
- new net N$65: R68.1, R69.2
- new net N$66: R69.1, R70.2
- new net N$67: R70.1, R71.2
- new net N$68: DISPLAY.P$3, R71.1, R72.2, R74.2
- new net N$69: EXTERNAL.19, IC5.7, R73.1
- new net N$7: IC1.3, R39.1
- new net N$70: R75.2, R76.1, R77.2
- new net N$71: IC5.6, R77.1
- new net N$72: IC5.5, R73.2, R74.1
- new net N$73: POT3.P$2, R60.2
- new net N$74: IC6.2, POT3.P$4
- new net N$75: POT3.P$1, R61.2
- new net N$76: C12.1, U$2.P$3
- new net N$77: C12.2, U$2.P$4
- new net N$78: C13.2, D12.A, OUT.P$3, R67.2, R81.2, U$2.P$5
- new net N$79: D11.C, D12.C
- new net N$80: R79.2, R80.1
- new net N$81: R82.1, R83.2
- new net N$82: R83.1, R84.1
- new net N$83: R80.2, R81.1
- new net N$84: D13.C, D14.C
- new net N$85: IC7.2, R87.1, R88.2
- new net N$86: IC7.3, R89.1
- new net N$87: R89.2, R90.2, R91.1
- new net N$88: IC7.1, IC8.8, R88.1
- new net N$89: R92.1, R93.2
- new net N$90: R93.1, R94.2
- new net N$91: R94.1, R95.2
- new net N$92: R95.1, R96.2
- new net N$93: DISPLAY.P$4, R96.1, R97.2, R99.2
- new net N$94: EXTERNAL.20, IC7.7, R98.1
- new net N$95: R100.2, R101.1, R102.2
- new net N$96: IC7.6, R102.1
- new net N$97: IC7.5, R98.2, R99.1
- new net N$98: POT4.P$2, R85.2
- new net N$99: IC8.2, POT4.P$4
- net +15V: now also IC1.8, IC10.4, IC11.8, IC12.4, IC13.8, IC14.4, IC15.8, IC16.4, IC4.4, IC5.8, IC6.4, IC7.8, IC8.4, IC9.8, R1.1, R101.2, R110.1, R116.2, R126.2, R135.1, R141.2, R151.2, R160.1, R166.2, R176.2, R185.1, R191.2, R201.2, R41.2, R51.2, R60.1, R66.2, R76.2, R85.1, R91.2; no longer IC4.8
- net +5V: now also IC10.5, IC12.5, IC14.5, IC16.5, IC4.5, IC6.5, IC8.5
- net -15V: now also IC1.4, IC10.7, IC11.4, IC12.7, IC13.4, IC14.7, IC15.4, IC16.7, IC4.7, IC5.4, IC6.7, IC7.4, IC8.7, IC9.4, R100.1, R111.1, R115.1, R125.1, R136.1, R140.1, R150.1, R161.1, R165.1, R175.1, R186.1, R190.1, R200.1, R36.1, R40.1, R50.1, R61.1, R65.1, R75.1, R86.1, R90.1; no longer IC4.4
- net GND: now also D1.A, D11.A, D15.A, D19.A, D23.A, D27.A, D31.A, IC10.3, IC12.3, IC14.3, IC16.3, IC4.3, IC6.3, IC8.3, R109.2, R122.1, R134.2, R147.1, R159.2, R172.1, R184.2, R197.1, R209.2, R47.1, R59.2, R72.1, R84.2, R97.1
- net MAN: now also IC10.6, IC12.6, IC14.6, IC16.6, IC4.6, IC6.6, IC8.6
- net N$35: now also IC2.7; no longer IC4.1
- net N$37: now also IC2.6; no longer IC4.3
- net N$39: now also IC2.5; no longer IC4.2
- net V+_SAFE: now also U$1.P$7, U$2.P$7, U$3.P$7, U$5.P$7, U$6.P$7, U$7.P$7, U$8.P$7
- net V-_SAFE: now also U$1.P$6, U$2.P$6, U$3.P$6, U$5.P$6, U$6.P$6, U$7.P$6, U$8.P$6
- net VIN+: now also D13.A, D17.A, D21.A, D25.A, D29.A, D33.A, D5.A, IC10.1, IC12.1, IC14.1, IC16.1, IC4.1, IC6.1, IC8.1, U$1.P$2, U$2.P$2, U$3.P$2, U$5.P$2, U$6.P$2, U$7.P$2, U$8.P$2
- net VIN-: now also C11.1, C13.1, C15.1, C17.1, C19.1, C21.1, C23.1, D14.A, D18.A, D22.A, D26.A, D30.A, D34.A, D6.A, R104.1, R107.2, R129.1, R132.2, R154.1, R157.2, R179.1, R182.2, R204.1, R207.2, R54.1, R57.2, R79.1, R82.2, U$1.P$1, U$2.P$1, U$3.P$1, U$5.P$1, U$6.P$1, U$7.P$1, U$8.P$1

Commit message: 8chan
Parts:
- R1, R110, R111, R124, R13, R135, R136, R14, R149, R160, R161, R174, R185, R186, R199, R28, R32, R36, R49, R60, R61, R74, R85, R86, R99: device rcl:0207/15 -> rcl:0207/10
- moved R199 56.6 mm to (88.4, 251.7)
- moved R201 56.5 mm to (28.4, 252.7)
- moved IC15 56.4 mm to (71.9, 250.7)
- moved IC16 56.4 mm to (55.6, 250.7)
- moved R189 56.4 mm to (49.5, 260.4)
- moved R191 56.4 mm to (39.4, 252.2)
- moved R198 56.4 mm to (75.7, 258.6)
- moved R202 56.4 mm to (68.3, 263.1)
- moved R187 56.4 mm to (82.5, 247.1)
- moved R188 56.4 mm to (65.5, 241.8)
- moved R190 56.4 mm to (44.5, 249.7)
- moved R200 56.4 mm to (33.8, 249.7)
- moved R32 53.4 mm to (21.1, 252.7), turned to 270 degrees
- moved R176 52.5 mm to (29.0, 220.0)
- moved IC13 52.3 mm to (71.4, 220.5)
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Routing:
- net V-_SAFE: track 0.00 -> 483.7 mm
- net V+_SAFE: track 0.00 -> 468.9 mm
- net +5V: track 0.00 -> 333.9 mm
- net -15V: track 0.00 -> 294.9 mm, vias 0 -> 1
- net +15V: track 0.00 -> 256.8 mm
- net V-: track 0.00 -> 112.7 mm
- net V+: track 0.00 -> 55.7 mm
- net N$19: track 0.00 -> 28.8 mm
- net N$10: track 0.00 -> 27.3 mm
- net N$17: track 0.00 -> 16.3 mm
- net N$2: track 0.00 -> 15.2 mm
- net N$5: track 0.00 -> 7.37 mm
- net MAN: track 0.00 -> 7.11 mm
- net N$1: track 0.00 -> 6.86 mm
- added copper zone on layer 1, net GND

Commit message: submit 8 chan
Parts:
- C8, C9: value cc -> 1n
- Q1, Q2: value 2N3906 -> STX616-AP
- R10, R12: value rb -> 1k
- R11, R8: value rlim -> 68
- R15, R9: value rl -> 4.99M
- T1, T2: value 2N3904 -> ZTX560
Routing:
- net VIN-: track 0.00 -> 888.5 mm, vias 0 -> 3
- net -15V: track 294.9 -> 1083.4 mm, vias 1 -> 7
- net VIN+: track 0.00 -> 760.8 mm, vias 0 -> 1
- net +15V: track 256.8 -> 848.9 mm, vias 0 -> 2
- net N$68: track 0.00 -> 472.4 mm, vias 0 -> 3
- net N$93: track 0.00 -> 462.2 mm, vias 0 -> 4
- net N$43: track 0.00 -> 426.8 mm, vias 0 -> 4
- net N$34: track 0.00 -> 375.7 mm, vias 0 -> 1
- net MAN: track 7.11 -> 380.1 mm, vias 0 -> 3
- net N$193: track 0.00 -> 366.4 mm, vias 0 -> 2
- net N$118: track 0.00 -> 347.6 mm, vias 0 -> 3
- net CMD1: track 0.00 -> 335.0 mm, vias 0 -> 3
- net N$143: track 0.00 -> 311.2 mm, vias 0 -> 5
- net N$35: track 0.00 -> 288.6 mm, vias 0 -> 4
- net N$44: track 0.00 -> 282.8 mm, vias 0 -> 1
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
Commit message: fix multichannel bugs
Parts:
- moved C3 14.2 mm to (190.2, 31.8), turned to 0 degrees
- moved HVIN 10.7 mm to (190.8, 11.2)
- moved D2 9.20 mm to (194.1, 23.9), turned to 0 degrees
Routing:
- net GND: track 0.00 -> 53.1 mm, vias 0 -> 5
- net V+: track 55.7 -> 33.4 mm
- net V-: track 112.7 -> 104.1 mm
Other:
- board size 215.9 x 292.1 mm -> 212.9 x 292.1 mm
